File: PCB/MCU.kicad_sch (KiCad schematic)
At the start: 12 parts, among them J1 TC2030-NL, U7 STM32G431C8Ux

Commit message: f
Parts:
- removed C1 (x2): 100n, symbol Device:C_Small
- removed R6 (x2): 1k, symbol Device:R_Small
- removed U7: STM32G431C8Ux, Package_DFN_QFN:QFN-48-1EP_7x7mm_P0.5mm_EP5.6x5.6mm, symbol MCU_ST_STM32G4:STM32G431C8Ux
- added C2 (x4): 100p, symbol Device:C_Small
- added L1: L_Small, symbol Device:L_Small
- added R13: 0m5, symbol Device:R_Small
- added R5 (x7): 10k, symbol Device:R_Small
- added R6 (x3): 1k5, symbol Device:R_Small
- added U4: STM32F051K6Ux, Package_DFN_QFN:QFN-32-1EP_5x5mm_P0.5mm_EP3.45x3.45mm, symbol MCU_ST_STM32F0:STM32F051K6Ux
- added U6: INA180A3, Package_TO_SOT_SMD:SOT-23-5, symbol Amplifier_Current:INA180A3
Connections:
- net +2V5 is gone; now on net +3V3_REF: C4.2
- net +3V3: now also L1.1, U4.1 (VDD), U4.17 (VDD)
- net +3V3_REF: now also L1.2, U4.5 (VDDA), U6.5 (V+)
- net BOOT0: now also U4.31 (BOOT0)
- net GND: now also C2.1, C2.1, C2.1, C2.1, R13.1, R6.1, R6.1, R6.1, U4.33 (VSS), U6.2 (GND), U6.4 (-)
- net HI_A: now also U4.20 (PA10)
- net HI_B: now also U4.19 (PA9)
- net HI_C: now also U4.18 (PA8)
- net LI_A: now also U4.15 (PB1)
- net LI_B: now also U4.14 (PB0)
- net LI_C: now also U4.13 (PA7)
- net RST: now also U4.4 (NRST)
- net SWC: now also U4.24 (PA14)
- net SWD: now also U4.23 (PA13)
- net V_Sen_A: now also C2.2, R5.1, R5.2, R6.2, U4.11 (PA5)
- net V_Sen_B: now also C2.2, R5.1, R5.2, R6.2, U4.10 (PA4)
- net V_Sen_C: now also C2.2, R5.1, R5.2, R6.2, U4.6 (PA0)
- net SWO: no longer names the net of J1.6 (SWO)
- new net: R5.2, U6.1
- new net GNDREF: R13.2, U6.3 (+)
- new net I_Sen: C2.2, R5.1, U4.8 (PA2)
- new net PWM_In: U4.27 (PB4)
- new net Phase_Out_A: R5.2
- new net Phase_Out_B: R5.2
- new net Phase_Out_C: R5.2
- new net USART_RX: U4.30 (PB7)
- new net USART_TX: U4.29 (PB6)
- new net V_Sen_Com: R5.1, R5.1, R5.1, U4.7 (PA1)
- no-connect marks 0 -> 12
Other:
- note added: "50A * 0.0005R * 100 = 2.5V"
- note added: "50A^2 * 0.0005R = 1.25W"
- note added: "ADC_IN2"
- note added: "COMP1_INM"
- note added: "COMP1_INP"
- note added: "Gain = 50"
- note added: "LPF BW = 159.24kHz"
- note added: "Max voltage (25.2V input) = 2.91V"
- note added: "TIM1_CH1"
- note added: "TIM1_CH1N"
- note added: "TIM1_CH2"
- note added: "TIM1_CH2N"
- note added: "TIM1_CH3"
- note added: "TIM1_CH3N"
- note added: "TIM3_CH1"
- note added: "Use kelvin connections to current sense resistor for best accuracy"
- note removed: "ADC1_IN1"
- note removed: "ADC1_IN2"
- note removed: "ADC1_IN3"
- note removed: "ADC1_IN4"
- note removed: "ADC2_IN13"
- note removed: "ADC2_IN17"
- note removed: "ADC2_IN3"
- moved on the sheet: C1, C18, C4, J1

Commit message: d
Parts:
- removed C4: 1u, symbol Device:C_Small
- removed J1: TC2030-NL, Connector:Tag-Connect_TC2030-IDC-NL_2x03_P1.27mm_Vertical, symbol Connector:Conn_ARM_SWD_TagConnect_TC2030-NL
- removed R5 (x3): 10k, symbol Device:R_Small
- added C22: 4u7, Ariamelon-Device:C_0603_1608Metric, symbol Device:C_Small
- added R21: 220, Ariamelon-Device:R_0402_1005Metric, symbol Device:R_Small
- added Y1: 8M, Crystal:Resonator_SMD_Murata_CSTxExxV-3Pin_3.0x1.1mm, symbol Device:Resonator_Small
- C19: renamed from C18; footprint (none) -> Ariamelon-Device:C_0603_1608Metric
- C20, C21: renamed from C1; footprint (none) -> Ariamelon-Device:C_0603_1608Metric
- C23, C28: renamed from C4; footprint (none) -> Ariamelon-Device:C_0603_1608Metric
- C24, C25, C26, C27: renamed from C2; footprint (none) -> Ariamelon-Device:C_0603_1608Metric
- R13, R14, R15, R19: renamed from R5; footprint (none) -> Ariamelon-Device:R_0402_1005Metric
- R16, R18, R20: renamed from R6; footprint (none) -> Ariamelon-Device:R_0402_1005Metric
- renumbered L1 to L4, R13 to R17, U6 to U5
Connections:
- net +3V3_REF: now also C22.2
- net GND: now also C22.1, Y1.2
- net I_Sen: now also U4.9 (PA3); no longer U4.8 (PA2)
- net PWM_In: now also U4.8 (PA2); no longer U4.27 (PB4)
- net V_Sen_A: now also C27.2, R15.1, R20.2, U4.10 (PA4), U4.12 (PA6); no longer U4.11 (PA5)
- net V_Sen_B: now also U4.11 (PA5); no longer U4.10 (PA4)
- net at U4.2 (PF0): now also Y1.1
- net at U4.3 (PF1): now also R21.1
- removed net V_Sen_C: C27.2, R15.1, R20.2, U4.6 (PA0)
- net V_Sen_Com: no longer names the net of U4.7 (PA1)
- new net: R21.2, Y1.3
- no-connect marks 12 -> 10
Other:
- note added: "ADC_IN3"
- note added: "ADC_IN4"
- note added: "ADC_IN5"
- note added: "ADC_IN6"
- note added: "TIM15_CH1 (Input Capture)"
- note added: "TIM1_CH1 (PWM)"
- note added: "TIM1_CH1N (PWM complementary)"
- note added: "TIM1_CH2 (PWM)"
- note added: "TIM1_CH2N (PWM complementary)"
- note added: "TIM1_CH3 (PWM)"
- note added: "TIM1_CH3N (PWM complementary)"
- note removed: "ADC_IN2"
- note removed: "COMP1_INM"
- note removed: "COMP1_INP"
- note removed: "TIM1_CH1"
- note removed: "TIM1_CH1N"
- note removed: "TIM1_CH2"
- note removed: "TIM1_CH2N"
- note removed: "TIM1_CH3"
- note removed: "TIM1_CH3N"
- note removed: "TIM3_CH1"
- moved on the sheet: C24, C25, C27, R16, R18, R20

Commit message: f
Parts:
- removed C22: 4u7, Ariamelon-Device:C_0603_1608Metric, symbol Device:C_Small
- added C1: 1u, Ariamelon-Device:C_0603_1608Metric, symbol Device:C_Small
Connections:
- net +3V3_REF: now also C1.2
- net GND: now also C1.1
- net I_Sen: now also U4.7 (PA1); no longer U4.9 (PA3)
- net PWM_In: now also U4.27 (PB4); no longer U4.8 (PA2)
- net V_Sen_A: now also U4.11 (PA5), U4.9 (PA3); no longer U4.10 (PA4), U4.12 (PA6)
- net V_Sen_B: now also U4.10 (PA4); no longer U4.11 (PA5)
- net USART_RX renamed USART1_RX
- net USART_TX renamed USART1_TX
- new net V_Sen_In: U4.8 (PA2)
- no-connect marks 10 -> 9
Other:
- note added: "ADC_IN1"
- note added: "ADC_IN2"
- note added: "TIM3_CH1 (Input Capture)"
- note removed: "ADC_IN6"
- note removed: "TIM15_CH1 (Input Capture)"
- moved on the sheet: C19, C20, C21, C23, C24, C25, C26, C27, C28, L4, R13, R14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

Commit message: f
Parts:
- removed C26: 100p, Ariamelon-Device:C_0603_1608Metric, symbol Device:C_Small
- removed C28: 1u, Ariamelon-Device:C_0603_1608Metric, symbol Device:C_Small
- removed R17: 0m5, symbol Device:R_Small
- removed R19: 10k, Ariamelon-Device:R_0402_1005Metric, symbol Device:R_Small
- removed U4: STM32F051K6Ux, Package_DFN_QFN:QFN-32-1EP_5x5mm_P0.5mm_EP3.45x3.45mm, symbol MCU_ST_STM32F0:STM32F051K6Ux
- removed U5: INA180A3, Package_TO_SOT_SMD:SOT-23-5, symbol Amplifier_Current:INA180A3
- added U4: STM32F051K6Tx, Package_QFP:LQFP-32_7x7mm_P0.8mm, symbol MCU_ST_STM32F0:STM32F051K6Tx
- renumbered C19 to C16, C20 to C17, C21 to C18, C23 to C20, C24 to C21, C25 to C23, C27 to C25, R21 to R19, R13 to R20, R14 to R21, R15 to R22, R16 to R24, R18 to R25, R20 to R27
Connections:
- net +3V3: now also U4.1 (VDD), U4.17 (VDD)
- net +3V3_REF: now also U4.5 (VDDA)
- net BOOT0: now also U4.31 (BOOT0)
- net GND: now also U4.16 (VSS), U4.32 (VSS)
- net HI_A: now also U4.18 (PA8)
- net HI_B: now also U4.19 (PA9)
- net HI_C: now also U4.20 (PA10)
- net I_Sen: now also U4.7 (PA1)
- net LI_A: now also U4.13 (PA7)
- net LI_B: now also U4.14 (PB0)
- net LI_C: now also U4.15 (PB1)
- net PWM_In: now also U4.27 (PB4)
- net RST: now also U4.4 (NRST)
- net SWC: now also U4.24 (PA14)
- net SWD: now also U4.23 (PA13)
- net USART1_RX: now also U4.30 (PB7)
- net USART1_TX: now also U4.29 (PB6)
- net V_Sen_A: now also U4.11 (PA5), U4.9 (PA3)
- net V_Sen_B: now also U4.10 (PA4)
- net V_Sen_In: now also U4.8 (PA2)
- net at Y1.1: now also U4.2 (PF0)
- net at R19.1: now also U4.3 (PF1)
- no-connect marks 9 -> 7
Other:
- note removed: "50A * 0.0005R * 100 = 2.5V"
- note removed: "50A^2 * 0.0005R = 1.25W"
- note removed: "Gain = 50"
- note removed: "Use kelvin connections to current sense resistor for best accuracy"
