File: PCB/MCU.kicad_sch (KiCad schematic)
At the start: 19 parts, among them U4 STM32F051K6Tx, U7 ATmega328P-P, Y1 8M

Commit message: Completed initial prototype.
Parts:
- removed C1: 1u, Ariamelon-Device:C_0603_1608Metric, symbol Device:C_Small
- removed C16: 4u7, Ariamelon-Device:C_0603_1608Metric, symbol Device:C_Small
- removed C17, C18: 100n, Ariamelon-Device:C_0603_1608Metric, symbol Device:C_Small
- removed C21, C23, C25: 100p, Ariamelon-Device:C_0603_1608Metric, symbol Device:C_Small
- removed L4: L_Small, symbol Device:L_Small
- removed U4: STM32F051K6Tx, Package_QFP:LQFP-32_7x7mm_P0.8mm, symbol MCU_ST_STM32F0:STM32F051K6Tx
- removed Y1: 8M, Crystal:Resonator_SMD_Murata_CSTxExxV-3Pin_3.0x1.1mm, symbol Device:Resonator_Small
- added C1 (x6): 10u, Ariamelon-Device:CP_Radial_D5.0mm_P2.54mm, symbol Device:C_Polarized_Small
- added C13, C15: 22p, Ariamelon-Device:C_Disc_D5.0mm_W2.5mm_P2.54mm, symbol Device:C_Small
- added C16, C7, C8, C9: 1000u, Ariamelon-Device:CP_Radial_D16.0mm_P7.62mm, symbol Device:C_Polarized_Small
- added C3: 100n, Ariamelon-Device:C_Disc_D6.0mm_W2.5mm_P5.08mm, symbol Device:C_Small
- added D7 (x3): 400x, Diode_THT:D_DO-35_SOD27_P7.62mm_Horizontal, symbol Device:D_Small
- added H1: VCC, Ariamelon-HolePad:MountingHole_3.2mm_M3_Pad, symbol Ariamelon-Misc:MountingHole_Pad
- added J1: Prog, Connector_PinSocket_2.54mm:PinSocket_1x04_P2.54mm_Vertical, symbol Connector_Generic:Conn_01x04
- added J2: Receiver, Connector_PinSocket_2.54mm:PinSocket_1x03_P2.54mm_Vertical, symbol Connector_Generic:Conn_01x03
- added J3: Bat_In, Connector_AMASS:AMASS_XT60-M_1x02_P7.20mm_Vertical, symbol Connector_Generic:Conn_01x02
- added R22: 4k7, Resistor_THT:R_Axial_DIN0204_L3.6mm_D1.6mm_P7.62mm_Horizontal, symbol Device:R_Small
- added R23: 560, Resistor_THT:R_Axial_DIN0204_L3.6mm_D1.6mm_P7.62mm_Horizontal, symbol Device:R_Small
- added R25: 10k, Resistor_THT:R_Axial_DIN0204_L3.6mm_D1.6mm_P7.62mm_Horizontal, symbol Device:R_Small
- added R32, R33, R34: 47k, Resistor_THT:R_Axial_DIN0204_L3.6mm_D1.6mm_P7.62mm_Horizontal, symbol Device:R_Small
- added SW1: RST, Button_Switch_THT:SW_PUSH_6mm, symbol Ariamelon-Switch:SW_Push_Small
- added SW2: Speed+, Button_Switch_THT:SW_PUSH_6mm, symbol Ariamelon-Switch:SW_Push_Small
- added SW3: Speed-, Button_Switch_THT:SW_PUSH_6mm, symbol Ariamelon-Switch:SW_Push_Small
- added U5: LM317, Package_TO_SOT_THT:TO-220-3_Vertical, symbol Regulator_Linear:LM317_TO-220
- added U6: LM7805, Package_TO_SOT_THT:TO-220-3_Vertical, symbol Regulator_Linear:L7805
- added Y1: 16M, Crystal:Crystal_HC49-4H_Vertical, symbol Device:Crystal_Small
- C20: value 10n -> 22p; footprint Ariamelon-Device:C_0603_1608Metric -> Ariamelon-Device:C_Disc_D5.0mm_W2.5mm_P2.54mm
- R19: value 220 -> 1; footprint Ariamelon-Device:R_0402_1005Metric -> Resistor_THT:R_Axial_DIN0204_L3.6mm_D1.6mm_P7.62mm_Horizontal
- R26: renamed from R20; value 10k -> 47k; footprint Ariamelon-Device:R_0402_1005Metric -> Resistor_THT:R_Axial_DIN0204_L3.6mm_D1.6mm_P7.62mm_Horizontal
- R27: renamed from R21; value 10k -> 47k; footprint Ariamelon-Device:R_0402_1005Metric -> Resistor_THT:R_Axial_DIN0204_L3.6mm_D1.6mm_P7.62mm_Horizontal
- R28: renamed from R22; value 10k -> 47k; footprint Ariamelon-Device:R_0402_1005Metric -> Resistor_THT:R_Axial_DIN0204_L3.6mm_D1.6mm_P7.62mm_Horizontal
- R29: renamed from R24; value 1k5 -> 4k7; footprint Ariamelon-Device:R_0402_1005Metric -> Resistor_THT:R_Axial_DIN0204_L3.6mm_D1.6mm_P7.62mm_Horizontal
- R30: renamed from R25; value 1k5 -> 4k7; footprint Ariamelon-Device:R_0402_1005Metric -> Resistor_THT:R_Axial_DIN0204_L3.6mm_D1.6mm_P7.62mm_Horizontal
- R31: renamed from R27; value 1k5 -> 4k7; footprint Ariamelon-Device:R_0402_1005Metric -> Resistor_THT:R_Axial_DIN0204_L3.6mm_D1.6mm_P7.62mm_Horizontal
- U4: renamed from U7; footprint Package_DIP:DIP-28_W7.62mm -> Package_DIP:DIP-28_W7.62mm_Socket
Connections:
- net +3V3_REF is gone; now on net PWM_In: C20.2
- net GND: now also U4.22 (GND), U4.8 (GND), C1.2, C1.2, C1.2, C1.2, C1.2, C1.2, C13.1, C15.1, C16.2, C3.2, C7.2, C8.2, C9.2, J1.4 (Pin_4), J2.1 (Pin_1), J3.1 (Pin_1), R22.1, SW1.2 (B), SW2.2 (B), SW3.2 (B), U6.2 (GND)
- net HI_A: now also U4.4 (PD2)
- net LI_A: now also U4.28 (PC5)
- net LI_B: now also U4.27 (PC4)
- net LI_C: now also U4.26 (PC3)
- net PWM_In: now also U4.14 (PB0), J2.3 (Pin_3)
- net RST: now also U4.1 (~{RESET}/PC6), C3.1, R25.2, SW1.1 (A)
- net V_Sen_A: now also U4.25 (PC2), R32.2; no longer R28.1, R31.2
- net V_Sen_B: now also U4.24 (PC1), R33.2
- net at R19.2: now also C1.1, D7.1 (K), U6.1 (IN)
- net +12V: now reaches R19.1
- net +12V: now also C16.1, D7.1 (K), D7.2 (A), R23.1, U5.2 (VO)
- net XTAL2: now reaches U4.10 (XTAL2/PB7)
- net XTAL2: now also C15.2, Y1.2
- net V_Sen_COM: now reaches U4.12 (PD6)
- net V_Sen_COM: now also R32.1, R33.1, R34.1
- net Speed+: now reaches U4.15 (PB1)
- net Speed+: now also SW2.1 (A)
- net Speed-: now reaches U4.16 (PB2)
- net Speed-: now also SW3.1 (A)
- net RX: now reaches U4.2 (PD0)
- net RX: now also J1.2 (Pin_2)
- net +5V: now reaches U4.20 (AVCC)
- net +5V: now also U4.21 (AREF), U4.7 (VCC), C1.1, C1.1, C1.1, D7.2 (A), J1.1 (Pin_1), J2.2 (Pin_2), R25.1, U6.3 (OUT)
- net V_Sen_C: now reaches U4.23 (PC0)
- net V_Sen_C: now also R28.1, R31.2, R34.2
- net TX: now reaches U4.3 (PD1)
- net TX: now also J1.3 (Pin_3)
- net XTAL1: now reaches U4.9 (XTAL1/PB6)
- net XTAL1: now also C13.2, Y1.1
- new net: C1.1, D7.2 (A), R22.2, R23.2, U5.1 (ADJ)
- new net VCC: C1.1, C7.1, C8.1, C9.1, D7.1 (K), H1.1, J3.2 (Pin_2), U5.3 (VI)
Other:
- note added: "-3dB point = 15.9kHz"
- note added: "16 bit PWM timer outputs"
- note added: "ADC0"
- note added: "ADC1"
- note added: "ADC2"
- note added: "AIN0"
- note added: "Comparator +ve input"
- note added: "Comparator -ve input"
- note added: "ICP1"
- note added: "Max voltage (25.2V input) = 2.01V"
- note added: "OC3A"
- note added: "OC4A"
- note added: "OC4B"
- note added: "Resistors must be 1% or better"
- note added: "Timer 1 input capture"
- note removed: "ADC_IN1"
- note removed: "ADC_IN2"
- note removed: "ADC_IN3"
- note removed: "ADC_IN4"
- note removed: "ADC_IN5"
- note removed: "LPF BW = 159.24kHz"
- note removed: "Max voltage (25.2V input) = 2.91V"
- note removed: "TIM1_CH1 (PWM)"
- note removed: "TIM1_CH1N (PWM complementary)"
- note removed: "TIM1_CH2 (PWM)"
- note removed: "TIM1_CH2N (PWM complementary)"
- note removed: "TIM1_CH3 (PWM)"
- note removed: "TIM1_CH3N (PWM complementary)"
- note removed: "TIM3_CH1 (Input Capture)"
- moved on the sheet: R26, R27, R28, R29, R30, R31, U4
