File: PCB/MCU.kicad_sch (KiCad schematic)
At the start: 19 parts, among them U4 STM32F051K6Tx, U7 ATmega328P-P, Y1 8M

Commit message: First draft of schematic done.
Parts:
- removed C1: 1u, Ariamelon-Device:C_0603_1608Metric, symbol Device:C_Small
- removed C16: 4u7, Ariamelon-Device:C_0603_1608Metric, symbol Device:C_Small
- removed C17, C18: 100n, Ariamelon-Device:C_0603_1608Metric, symbol Device:C_Small
- removed C20: 10n, Ariamelon-Device:C_0603_1608Metric, symbol Device:C_Small
- removed C21, C23: 100p, Ariamelon-Device:C_0603_1608Metric, symbol Device:C_Small
- removed L4: L_Small, symbol Device:L_Small
- removed U4: STM32F051K6Tx, Package_QFP:LQFP-32_7x7mm_P0.8mm, symbol MCU_ST_STM32F0:STM32F051K6Tx
- removed Y1: 8M, Crystal:Resonator_SMD_Murata_CSTxExxV-3Pin_3.0x1.1mm, symbol Device:Resonator_Small
- added C1 (x5): 10u, Capacitor_THT:C_Disc_D6.0mm_W2.5mm_P5.00mm, symbol Device:C_Small
- added C13: 1000u, Capacitor_THT:CP_Radial_D16.0mm_P7.50mm, symbol Device:C_Polarized_Small
- added C27, C28: 22p, Capacitor_THT:C_Disc_D5.0mm_W2.5mm_P2.50mm, symbol Device:C_Small
- added C3 (x3): 100n, Capacitor_THT:C_Disc_D6.0mm_W2.5mm_P5.00mm, symbol Device:C_Small
- added C3: 1u, Capacitor_THT:C_Disc_D6.0mm_W2.5mm_P5.00mm, symbol Device:C_Small
- added D7 (x3): 400x, Diode_THT:D_DO-41_SOD81_P7.62mm_Horizontal, symbol Device:D_Small
- added J1: Prog, Connector_PinSocket_2.54mm:PinSocket_1x04_P2.54mm_Vertical, symbol Connector_Generic:Conn_01x04
- added J2: Receiver, Connector_PinSocket_2.54mm:PinSocket_1x03_P2.54mm_Vertical, symbol Connector_Generic:Conn_01x03
- added J3: ICSP, Connector_PinSocket_2.54mm:PinSocket_2x03_P2.54mm_Vertical, symbol Connector_Generic:Conn_02x03_Odd_Even
- added R22: 4k7, Resistor_THT:R_Axial_DIN0207_L6.3mm_D2.5mm_P7.62mm_Horizontal, symbol Device:R_Small
- added R23: 560, Resistor_THT:R_Axial_DIN0207_L6.3mm_D2.5mm_P7.62mm_Horizontal, symbol Device:R_Small
- added R25, R26, R27: 10k, Resistor_THT:R_Axial_DIN0207_L6.3mm_D2.5mm_P7.62mm_Horizontal, symbol Device:R_Small
- added R34, R35, R36: 47k, Resistor_THT:R_Axial_DIN0207_L6.3mm_D2.5mm_P7.62mm_Horizontal, symbol Device:R_Small
- added SW1: RST, Button_Switch_THT:SW_PUSH_6mm, symbol Ariamelon-Switch:SW_Push_Small
- added SW2: Speed+, Button_Switch_THT:SW_PUSH_6mm, symbol Ariamelon-Switch:SW_Push_Small
- added SW3: Speed-, Button_Switch_THT:SW_PUSH_6mm, symbol Ariamelon-Switch:SW_Push_Small
- added U5: LM317, Package_TO_SOT_THT:TO-220-3_Vertical, symbol Regulator_Linear:LM317_TO-220
- added U6: LM7805, Package_TO_SOT_THT:TO-220-3_Vertical, symbol Regulator_Linear:L7805
- added Y1: 16M, Crystal:Crystal_HC49-U_Vertical, symbol Device:Crystal_Small
- C25: value 100p -> 22p; footprint Ariamelon-Device:C_0603_1608Metric -> Capacitor_THT:C_Disc_D6.0mm_W2.5mm_P5.00mm
- R19: value 220 -> 10; footprint Ariamelon-Device:R_0402_1005Metric -> Resistor_THT:R_Axial_DIN0207_L6.3mm_D2.5mm_P7.62mm_Horizontal
- R28: renamed from R20; value 10k -> 47k; footprint Ariamelon-Device:R_0402_1005Metric -> Resistor_THT:R_Axial_DIN0207_L6.3mm_D2.5mm_P7.62mm_Horizontal
- R29: renamed from R21; value 10k -> 47k; footprint Ariamelon-Device:R_0402_1005Metric -> Resistor_THT:R_Axial_DIN0207_L6.3mm_D2.5mm_P7.62mm_Horizontal
- R30: renamed from R22; value 10k -> 47k; footprint Ariamelon-Device:R_0402_1005Metric -> Resistor_THT:R_Axial_DIN0207_L6.3mm_D2.5mm_P7.62mm_Horizontal
- R31: renamed from R24; value 1k5 -> 4k7; footprint Ariamelon-Device:R_0402_1005Metric -> Resistor_THT:R_Axial_DIN0207_L6.3mm_D2.5mm_P7.62mm_Horizontal
- R32: renamed from R25; value 1k5 -> 4k7; footprint Ariamelon-Device:R_0402_1005Metric -> Resistor_THT:R_Axial_DIN0207_L6.3mm_D2.5mm_P7.62mm_Horizontal
- R33: renamed from R27; value 1k5 -> 4k7; footprint Ariamelon-Device:R_0402_1005Metric -> Resistor_THT:R_Axial_DIN0207_L6.3mm_D2.5mm_P7.62mm_Horizontal
- renumbered U7 to U4
Connections:
- net GND: now also U4.22 (GND), U4.8 (GND), C1.1, C1.1, C1.1, C1.1, C1.1, C13.2, C27.1, C28.1, C3.2, C3.2, C3.2, C3.2, J1.4 (Pin_4), J2.1 (Pin_1), J3.6 (Pin_6), R22.1, SW1.2 (B), SW2.2 (B), SW3.2 (B), U6.2 (GND)
- net HI_C: now also U4.4 (PD2)
- net LI_A: now also U4.26 (PC3)
- net LI_B: now also U4.27 (PC4)
- net LI_C: now also U4.28 (PC5)
- net PWM_In: now also C25.2, U4.14 (PB0), J2.3 (Pin_3)
- net RST: now also U4.1 (~{RESET}/PC6), C3.1, J3.5 (Pin_5), R25.2, SW1.1 (A)
- net V_Sen_A: now also U4.23 (PC0), R34.2; no longer C25.2, R30.1, R33.2
- net V_Sen_B: now also U4.24 (PC1), R35.2
- net at R19.2: now also C1.2, D7.1 (K), U6.1 (IN)
- net +12V: now reaches R19.1
- net +12V: now also C1.2, C1.2, D7.1 (K), D7.2 (A), D7.2 (A), R23.1, U5.2 (VO)
- net XTAL2: now reaches U4.10 (XTAL2/PB7)
- net XTAL2: now also C28.2, Y1.2
- net V_Sen_COM: now reaches U4.12 (PD6)
- net V_Sen_COM: now also R34.1, R35.1, R36.1
- net Speed+: now reaches U4.15 (PB1)
- net Speed+: now also C3.1, R26.2, SW2.1 (A)
- net Speed-: now reaches U4.16 (PB2)
- net Speed-: now also C3.1, R27.2, SW3.1 (A)
- net MOSI: now reaches U4.17 (PB3)
- net MOSI: now also J3.4 (Pin_4)
- net MISO: now reaches U4.18 (PB4)
- net MISO: now also J3.1 (Pin_1)
- net SCK: now reaches U4.19 (PB5)
- net SCK: now also J3.3 (Pin_3)
- net RX: now reaches U4.2 (PD0)
- net RX: now also J1.3 (Pin_3)
- net +5V: now reaches U4.20 (AVCC)
- net +5V: now also U4.21 (AREF), U4.7 (VCC), C1.2, C1.2, D7.2 (A), J1.1 (Pin_1), J2.2 (Pin_2), J3.2 (Pin_2), R25.1, R26.1, R27.1, U6.3 (OUT)
- net V_Sen_C: now reaches U4.25 (PC2)
- net V_Sen_C: now also R30.1, R33.2, R36.2
- net TX: now reaches U4.3 (PD1)
- net TX: now also J1.2 (Pin_2)
- net XTAL1: now reaches U4.9 (XTAL1/PB6)
- net XTAL1: now also C27.2, Y1.1
- new net: R22.2, R23.2, U5.1 (ADJ)
- new net VCC: C13.1, C3.1, D7.1 (K), U5.3 (VI)
- no-connect marks 7 -> 4
Other:
- note added: "-3dB point = 1.59kHz"
- note added: "16 bit PWM timer outputs"
- note added: "ADC0"
- note added: "ADC1"
- note added: "ADC2"
- note added: "AIN0"
- note added: "Comparator +ve input"
- note added: "Comparator -ve input"
- note added: "ICP1"
- note added: "Max voltage (25.2V input) = 2.01V"
- note added: "OC3A"
- note added: "OC4A"
- note added: "OC4B"
- note added: "Resistors must be 1% or better"
- note added: "Timer 1 input capture"
- note removed: "ADC_IN1"
- note removed: "ADC_IN2"
- note removed: "ADC_IN3"
- note removed: "ADC_IN4"
- note removed: "ADC_IN5"
- note removed: "LPF BW = 159.24kHz"
- note removed: "Max voltage (25.2V input) = 2.91V"
- note removed: "TIM1_CH1 (PWM)"
- note removed: "TIM1_CH1N (PWM complementary)"
- note removed: "TIM1_CH2 (PWM)"
- note removed: "TIM1_CH2N (PWM complementary)"
- note removed: "TIM1_CH3 (PWM)"
- note removed: "TIM1_CH3N (PWM complementary)"
- note removed: "TIM3_CH1 (Input Capture)"
- moved on the sheet: R28, R29, R30, R31, R32, R33, U4

Commit message: 28/10/2023 update
Began initial PCB layout.
Parts:
- removed C1: 10u, Capacitor_THT:C_Disc_D6.0mm_W2.5mm_P5.00mm, symbol Device:C_Small
- removed C3: 1u, Capacitor_THT:C_Disc_D6.0mm_W2.5mm_P5.00mm, symbol Device:C_Small
- removed J3: ICSP, Connector_PinSocket_2.54mm:PinSocket_2x03_P2.54mm_Vertical, symbol Connector_Generic:Conn_02x03_Odd_Even
- added C1: 10u, Ariamelon-Device:CP_Radial_D5.0mm_P2.54mm, symbol Device:C_Polarized_Small
- C1: footprint Capacitor_THT:C_Disc_D6.0mm_W2.5mm_P5.00mm -> Ariamelon-Device:CP_Radial_D5.0mm_P2.54mm; symbol Device:C_Small -> Device:C_Polarized_Small
- C13: footprint Capacitor_THT:CP_Radial_D16.0mm_P7.50mm -> Ariamelon-Device:CP_Radial_D16.0mm_P7.62mm
- C14: renamed from C27; footprint Capacitor_THT:C_Disc_D5.0mm_W2.5mm_P2.50mm -> Ariamelon-Device:C_Disc_D5.0mm_W2.5mm_P2.54mm
- C15: renamed from C28; footprint Capacitor_THT:C_Disc_D5.0mm_W2.5mm_P2.50mm -> Ariamelon-Device:C_Disc_D5.0mm_W2.5mm_P2.54mm
- C21: renamed from C25; footprint Capacitor_THT:C_Disc_D6.0mm_W2.5mm_P5.00mm -> Ariamelon-Device:C_Disc_D5.0mm_W2.5mm_P2.54mm
- C3: footprint Capacitor_THT:C_Disc_D6.0mm_W2.5mm_P5.00mm -> Ariamelon-Device:C_Disc_D6.0mm_W2.5mm_P5.08mm
- D7: footprint Diode_THT:D_DO-41_SOD81_P7.62mm_Horizontal -> Diode_THT:D_DO-35_SOD27_P7.62mm_Horizontal
- R19: value 10 -> 1; footprint Resistor_THT:R_Axial_DIN0207_L6.3mm_D2.5mm_P7.62mm_Horizontal -> Resistor_THT:R_Axial_DIN0204_L3.6mm_D1.6mm_P7.62mm_Horizontal
- R22, R23, R25, R26, R27, R28, R29, R30, R31, R32, R33, R34, R35, R36: footprint Resistor_THT:R_Axial_DIN0207_L6.3mm_D2.5mm_P7.62mm_Horizontal -> Resistor_THT:R_Axial_DIN0204_L3.6mm_D1.6mm_P7.62mm_Horizontal
- U4: footprint Package_DIP:DIP-28_W7.62mm -> Package_DIP:DIP-28_W7.62mm_Socket
- Y1: footprint Crystal:Crystal_HC49-U_Vertical -> Crystal:Crystal_HC49-4H_Vertical
Connections:
- net +12V: now also C13.1; no longer C1.2, D7.2 (A)
- net +5V: now also C1.1, C1.1; no longer C1.2, C1.2
- net GND: now also C1.2, C1.2, C1.2, C1.2, C1.2; no longer C1.1, C1.1, C1.1, C1.1
- net LI_A: now also U4.28 (PC5); no longer U4.26 (PC3)
- net LI_C: now also U4.26 (PC3); no longer U4.28 (PC5)
- net RX: now also J1.2 (Pin_2); no longer J1.3 (Pin_3)
- net TX: now also J1.3 (Pin_3); no longer J1.2 (Pin_2)
- net VCC: now also C1.1; no longer C13.1
- net V_Sen_A: now also U4.25 (PC2); no longer U4.23 (PC0)
- net V_Sen_C: now also U4.23 (PC0); no longer U4.25 (PC2)
- net at D7.1 (K), R19.2, U6.1 (IN): now also C1.1; no longer C1.2
- net at R22.2, R23.2, U5.1 (ADJ): now also C1.1, D7.2 (A)
- net HI_C renamed HI_A
- net MISO: no longer names the net of U4.18 (PB4)
- net MOSI: no longer names the net of U4.17 (PB3)
- net SCK: no longer names the net of U4.19 (PB5)
- no-connect marks 4 -> 7
Other:
- note added: "-3dB point = 15.9kHz"
- note removed: "-3dB point = 1.59kHz"
- moved on the sheet: D7, R19, R23, R28, R29, R30, R31, R33, R34, R35, R36, U6

Commit message: 30/10/2023 update
Completed initial PCB layout.
Parts:
- removed C3 (x2): 100n, Ariamelon-Device:C_Disc_D6.0mm_W2.5mm_P5.08mm, symbol Device:C_Small
- removed R26, R27: 10k, Resistor_THT:R_Axial_DIN0204_L3.6mm_D1.6mm_P7.62mm_Horizontal, symbol Device:R_Small
- added C1: 10u, Ariamelon-Device:CP_Radial_D5.0mm_P2.54mm, symbol Device:C_Polarized_Small
- added C7, C8, C9: 1000u, Ariamelon-Device:CP_Radial_D16.0mm_P7.62mm, symbol Device:C_Polarized_Small
- added H1: VCC, Ariamelon-HolePad:MountingHole_3.2mm_M3_Pad, symbol Ariamelon-Misc:MountingHole_Pad
- added J3: Bat_In, Connector_AMASS:AMASS_XT60-M_1x02_P7.20mm_Vertical, symbol Connector_Generic:Conn_01x02
- renumbered C14 to C13, C13 to C16, C21 to C20, R28 to R26, R29 to R27, R30 to R28, R31 to R29, R32 to R30, R33 to R31, R34 to R32, R35 to R33, R36 to R34
Connections:
- net +5V: now also C1.1
- net GND: now also C1.2, C7.2, C8.2, C9.2, J3.1 (Pin_1)
- net VCC: now also C7.1, C8.1, C9.1, H1.1, J3.2 (Pin_2)
Other:
- moved on the sheet: C1, C16, C20, D7, J1, J2, R19, R22, R23, R26, R27, R28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

Commit message: Fixed pin assignment. Added tentative arduino code.
Parts:
- removed H1: VCC, Ariamelon-HolePad:MountingHole_3.2mm_M3_Pad, symbol Ariamelon-Misc:MountingHole_Pad
- C16: value 1000u -> 470u; footprint Ariamelon-Device:CP_Radial_D16.0mm_P7.62mm -> Capacitor_THT:CP_Radial_D10.0mm_P5.00mm
- J1: footprint Connector_PinSocket_2.54mm:PinSocket_1x04_P2.54mm_Vertical -> Connector_PinHeader_2.54mm:PinHeader_1x04_P2.54mm_Vertical
- J2: footprint Connector_PinSocket_2.54mm:PinSocket_1x03_P2.54mm_Vertical -> Connector_PinHeader_2.54mm:PinHeader_1x03_P2.54mm_Vertical
- renumbered C1 to C10, C1 to C11, C1 to C12, C1 to C14, C3 to C17, C1 to C18, C1 to C19, D7 to D19, D7 to D20, D7 to D21, R19 to R24
Connections:
- net GND: now also J2.3 (Pin_3); no longer J2.1 (Pin_1)
- net HI_A: now also U4.17 (PB3); no longer U4.4 (PD2)
- net LI_A: now also U4.25 (PC2); no longer U4.28 (PC5)
- net LI_B: now also U4.24 (PC1); no longer U4.27 (PC4)
- net LI_C: now also U4.23 (PC0); no longer U4.26 (PC3)
- net PWM_In: now also J2.1 (Pin_1); no longer J2.3 (Pin_3)
- net Speed+: now also SW3.1 (A), U4.5 (PD3); no longer SW2.1 (A), U4.15 (PB1)
- net Speed-: now also SW2.1 (A), U4.4 (PD2); no longer SW3.1 (A), U4.16 (PB2)
- net V_Sen_A: now also U4.28 (PC5); no longer U4.25 (PC2)
- net V_Sen_B: now also U4.27 (PC4); no longer U4.24 (PC1)
- net V_Sen_C: now also U4.26 (PC3); no longer U4.23 (PC0)
- new net HI_B: U4.16 (PB2)
- new net HI_C: U4.15 (PB1)
- no-connect marks 7 -> 5
Other:
- note added: "ADC3"
- note added: "ADC4"
- note added: "ADC5"
- note added: "OC1A"
- note added: "OC1B"
- note added: "OC2A"
- note added: "PCINT0"
- note added: "PWM timer outputs"
- note added: "RC controller input"
- note removed: "16 bit PWM timer outputs"
- note removed: "ADC0"
- note removed: "ADC1"
- note removed: "ADC2"
- note removed: "ICP1"
- note removed: "OC3A"
- note removed: "OC4A"
- note removed: "OC4B"
- note removed: "Timer 1 input capture"
- moved on the sheet: J2

Commit message: V2 started
Parts:
- removed J3: Bat_In, Connector_AMASS:AMASS_XT60-M_1x02_P7.20mm_Vertical, symbol Connector_Generic:Conn_01x02
- removed R24: 1, Resistor_THT:R_Axial_DIN0204_L3.6mm_D1.6mm_P7.62mm_Horizontal, symbol Device:R_Small
- removed R26, R27, R28, R32, R33, R34: 47k, Resistor_THT:R_Axial_DIN0204_L3.6mm_D1.6mm_P7.62mm_Horizontal, symbol Device:R_Small
- removed R29, R30, R31: 4k7, Resistor_THT:R_Axial_DIN0204_L3.6mm_D1.6mm_P7.62mm_Horizontal, symbol Device:R_Small
- removed U4: ATmega328P-P, Package_DIP:DIP-28_W7.62mm_Socket, symbol MCU_Microchip_ATmega:ATmega328P-P
- removed U6: LM7805, Package_TO_SOT_THT:TO-220-3_Vertical, symbol Regulator_Linear:L7805
- added C10, C12: 100n, Ariamelon-Device:C_0603_1608Metric, symbol Device:C_Small
- added J7: Bat+, Ariamelon-HolePad:MountingHole_3.2mm_M3_Pad, symbol Connector_Generic:Conn_01x01
- added J8: Bat-, Ariamelon-HolePad:MountingHole_3.2mm_M3_Pad, symbol Connector_Generic:Conn_01x01
- added U4: ATmega328P-A, Package_QFP:TQFP-32_7x7mm_P0.8mm, symbol MCU_Microchip_ATmega:ATmega328P-A
- added U6: L78L05, Package_TO_SOT_SMD:SOT-89-3, symbol Regulator_Linear:L78L05_SOT89
- C14: renamed from C11; footprint Ariamelon-Device:CP_Radial_D5.0mm_P2.54mm -> Ariamelon-Device:C_0805_2012Metric; symbol Device:C_Polarized_Small -> Device:C_Small
- C15: renamed from C13; footprint Ariamelon-Device:C_Disc_D5.0mm_W2.5mm_P2.54mm -> Ariamelon-Device:C_0603_1608Metric
- C16: renamed from C15; footprint Ariamelon-Device:C_Disc_D5.0mm_W2.5mm_P2.54mm -> Ariamelon-Device:C_0603_1608Metric
- C17: renamed from C14; footprint Ariamelon-Device:CP_Radial_D5.0mm_P2.54mm -> Ariamelon-Device:C_0805_2012Metric; symbol Device:C_Polarized_Small -> Device:C_Small
- C18: renamed from C16; value 470u -> 10u; footprint Capacitor_THT:CP_Radial_D10.0mm_P5.00mm -> Ariamelon-Device:C_0805_2012Metric; symbol Device:C_Polarized_Small -> Device:C_Small
- C19: renamed from C18; footprint Ariamelon-Device:CP_Radial_D5.0mm_P2.54mm -> Ariamelon-Device:C_0805_2012Metric; symbol Device:C_Polarized_Small -> Device:C_Small
- C20: renamed from C17; footprint Ariamelon-Device:C_Disc_D6.0mm_W2.5mm_P5.08mm -> Ariamelon-Device:C_0603_1608Metric
- C21: renamed from C19; footprint Ariamelon-Device:CP_Radial_D5.0mm_P2.54mm -> Ariamelon-Device:C_0805_2012Metric; symbol Device:C_Polarized_Small -> Device:C_Small
- C22: renamed from C20; footprint Ariamelon-Device:C_Disc_D5.0mm_W2.5mm_P2.54mm -> Ariamelon-Device:C_0603_1608Metric
- C7: renamed from C10; footprint Ariamelon-Device:CP_Radial_D5.0mm_P2.54mm -> Ariamelon-Device:C_0805_2012Metric; symbol Device:C_Polarized_Small -> Device:C_Small
- C8: renamed from C12; value 10u -> 100n; footprint Ariamelon-Device:CP_Radial_D5.0mm_P2.54mm -> Ariamelon-Device:C_0603_1608Metric; symbol Device:C_Polarized_Small -> Device:C_Small
- D1: renamed from D19; footprint Diode_THT:D_DO-35_SOD27_P7.62mm_Horizontal -> Diode_SMD:D_SOD-123F
- D2: renamed from D20; footprint Diode_THT:D_DO-35_SOD27_P7.62mm_Horizontal -> Diode_SMD:D_SOD-123F
- D3: renamed from D21; footprint Diode_THT:D_DO-35_SOD27_P7.62mm_Horizontal -> Diode_SMD:D_SOD-123F
- J9: renamed from J1; footprint Connector_PinHeader_2.54mm:PinHeader_1x04_P2.54mm_Vertical -> Connector_PinHeader_2.54mm:PinHeader_1x06_P2.54mm_Vertical; symbol Connector_Generic:Conn_01x04 -> Connector_Generic:Conn_01x06
- R16: renamed from R22; value 4k7 -> 10k; footprint Resistor_THT:R_Axial_DIN0204_L3.6mm_D1.6mm_P7.62mm_Horizontal -> Ariamelon-Device:R_0603_1608Metric
- R17: renamed from R23; footprint Resistor_THT:R_Axial_DIN0204_L3.6mm_D1.6mm_P7.62mm_Horizontal -> Ariamelon-Device:R_0603_1608Metric
- R18: renamed from R25; footprint Resistor_THT:R_Axial_DIN0204_L3.6mm_D1.6mm_P7.62mm_Horizontal -> Ariamelon-Device:R_0603_1608Metric
- Y1: footprint Crystal:Crystal_HC49-4H_Vertical -> Crystal:Crystal_SMD_3225-4Pin_3.2x2.5mm; symbol Device:Crystal_Small -> Device:Crystal_GND24_Small
- renumbered C8 to C11, C9 to C13, C7 to C9, J2 to J10
Connections:
- net +12V: now also C19.1, D3.1 (K), U6.3 (IN)
- net +5V: now also J9.3 (Pin_3), C10.1, C12.1, U4.18 (AVCC), U4.20 (AREF), U4.4 (VCC), U4.6 (VCC), U6.1 (OUT); no longer J9.1 (Pin_1)
- net GND: now also J9.1 (Pin_1), J9.2 (Pin_2), Y1.2, Y1.4, C10.2, C12.2, J8.1 (Pin_1), U4.21 (GND), U4.3 (GND), U4.5 (GND), U6.2 (GND); no longer J9.4 (Pin_4)
- net HI_A: now also U4.15 (PB3)
- net HI_B: now also U4.14 (PB2)
- net HI_C: now also U4.13 (PB1)
- net LI_A: now also U4.25 (PC2)
- net LI_B: now also U4.24 (PC1)
- net LI_C: now also U4.23 (PC0)
- net PWM_In: now also U4.17 (PB5)
- net RST: now also U4.29 (~{RESET}/PC6)
- net RX: now also J9.4 (Pin_4), U4.30 (PD0); no longer J9.2 (Pin_2)
- net Speed+: now also U4.2 (PD4)
- net Speed-: now also U4.1 (PD3)
- net TX: now also J9.5 (Pin_5), U4.31 (PD1); no longer J9.3 (Pin_3)
- net VCC: now also J7.1 (Pin_1)
- net V_Sen_A: now also U4.28 (PC5)
- net V_Sen_B: now also U4.27 (PC4)
- net V_Sen_C: now also U4.26 (PC3)
- net V_Sen_COM: now also U4.10 (PD6)
- net XTAL1: now also U4.7 (XTAL1/PB6)
- net XTAL2: now also Y1.3, U4.8 (XTAL2/PB7); no longer Y1.2
- new net DTR: J9.6 (Pin_6)
- no-connect marks 5 -> 6
Other:
- moved on the sheet: C11, C13, C15, C16, C20, C22, C9, D1, D2, D3, J10, R16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

Commit message: f
Parts:
- removed C11, C13, C9: 1000u, Ariamelon-Device:CP_Radial_D16.0mm_P7.62mm, symbol Device:C_Polarized_Small
- removed C14, C17, C18, C19, C21: 10u, Ariamelon-Device:C_0805_2012Metric, symbol Device:C_Small
- removed D1, D2, D3: 400x, Diode_SMD:D_SOD-123F, symbol Device:D_Small
- removed R16: 10k, Ariamelon-Device:R_0603_1608Metric, symbol Device:R_Small
- removed R17: 560, Ariamelon-Device:R_0603_1608Metric, symbol Device:R_Small
- removed U5: LM317, Package_TO_SOT_THT:TO-220-3_Vertical, symbol Regulator_Linear:LM317_TO-220
- removed U6: L78L05, Package_TO_SOT_SMD:SOT-89-3, symbol Regulator_Linear:L78L05_SOT89
Other:
- note removed: "-3dB point = 15.9kHz"
- note removed: "Max voltage (25.2V input) = 2.01V"
- note removed: "Resistors must be 1% or better"
- moved on the sheet: C10, C12, C15, C16, C20, C22, C7, C8, J10, J7, J8, J9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
