File: PCB/PSU.kicad_sch (KiCad schematic)
At the start: 0 parts

Commit message: f
Parts:
- added U6: TPS62933, Package_TO_SOT_SMD:SOT-583-8, symbol Regulator_Switching:TPS62933
Connections:
- net VCC: now also U6.2 (EN), U6.3 (VIN)
- new net GND: U6.4 (GND)
Changed lines of the file:
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@@
 (kicad_sch (version 20230121) (generator eeschema)
   (paper "A4")
-  (symbol (lib_id "power:VCC") (at 71.12 50.8 0) (unit 1)
+  (junction (at 83.82 58.42) (diameter 0) (color 0 0 0 0)
+  )
+  (wire (pts (xy 83.82 55.88) (xy 83.82 58.42))
+    (stroke (width 0) (type default))
+  )
+  (wire (pts (xy 86.36 60.96) (xy 83.82 60.96))
+    (stroke (width 0) (type default))
+  )
+  (wire (pts (xy 83.82 60.96) (xy 83.82 58.42))
+    (stroke (width 0) (type default))
+  )
+  (wire (pts (xy 93.98 81.28) (xy 93.98 78.74))
+    (stroke (width 0) (type default))
+  )
+  (wire (pts (xy 83.82 58.42) (xy 86.36 58.42))
+    (stroke (width 0) (type default))
+  )
+  (symbol (lib_id "Regulator_Switching:TPS62933") (at 93.98 66.04 0) (unit 1)
     (in_bom yes) (on_board yes) (dnp no) (fields_autoplaced)
-    (property "Reference" "#PWR01" (at 71.12 54.61 0)
+    (property "Reference" "U6" (at 93.98 51.7357 0)
+      (effects (font (size 1.27 1.27)))
+    )
+    (property "Value" "TPS62933" (at 93.98 54.1599 0)
+      (effects (font (size 1.27 1.27)))
+    )
+    (property "Footprint" "Package_TO_SOT_SMD:SOT-583-8" (at 93.98 91.44 0)
       (effects (font (size 1.27 1.27)) hide)
     )
-    (property "Value" "VCC" (at 71.12 46.6669 0)
+    (property "Datasheet" "https://www.ti.com/lit/ds/symlink/tps62933.pdf" (at 93.98 88.9 0)
+      (effects (font (size 1.27 1.27)) hide)
+    )
+    (pin "1")
+    (pin "2")
+    (pin "3")
+    (pin "4")
+    (pin "5")
+    (pin "6")
+    (pin "7")
+    (pin "8")
+    (instances
+      (project "BLDC-Controller"
+        (path "/3f98b8cc-f1be-42b2-9c23-c425b8147bc0/69c4c952-9785-4038-8411-bd74bb4cf876"
+          (reference "U6") (unit 1)
+        )
+      )
+    )
+  )
+  (symbol (lib_id "power:VCC") (at 83.82 55.88 0) (unit 1)
+    (in_bom yes) (on_board yes) (dnp no) (fields_autoplaced)
+    (property "Reference" "#PWR01" (at 83.82 59.69 0)
+      (effects (font (size 1.27 1.27)) hide)
+    )
+    (property "Value" "VCC" (at 83.82 51.7469 0)
       (effects (font (size 1.27 1.27)))
     )
-    (property "Footprint" "" (at 71.12 50.8 0)
+    (property "Footprint" "" (at 83.82 55.88 0)
       (effects (font (size 1.27 1.27)) hide)
     )
-    (property "Datasheet" "" (at 71.12 50.8 0)
+    (property "Datasheet" "" (at 83.82 55.88 0)
       (effects (font (size 1.27 1.27)) hide)
     )
@@
     (instances
       (project "BLDC-Controller"
-        (path "/3f98b8cc-f1be-42b2-9c23-c425b8147bc0/66b89077-47c3-4560-995d-b73f8131e889"
-          (reference "#PWR01") (unit 1)
-        )
-        (path "/3f98b8cc-f1be-42b2-9c23-c425b8147bc0/03610141-8a53-451a-9aef-b28319aeb056"
-          (reference "#PWR015") (unit 1)
-        )
-        (path "/3f98b8cc-f1be-42b2-9c23-c425b8147bc0/40e3f309-d611-4837-a833-299126044f7d"
-          (reference "#PWR027") (unit 1)
-        )
         (path "/3f98b8cc-f1be-42b2-9c23-c425b8147bc0/69c4c952-9785-4038-8411-bd74bb4cf876"
           (reference "#PWR018") (unit 1)
         )
       )
+    )
+  )
+  (symbol (lib_id "power:GND") (at 93.98 81.28 0) (unit 1)
+    (in_bom yes) (on_board yes) (dnp no)
+    (property "Reference" "#PWR049" (at 93.98 87.63 0)
+      (effects (font (size 1.27 1.27)) hide)
+    )
+    (property "Value" "GND" (at 93.98 85.09 0)
+      (effects (font (size 1.27 1.27)) hide)
+    )
+    (property "Footprint" "" (at 93.98 81.28 0)
+      (effects (font (size 1.27 1.27)) hide)
+    )
+    (property "Datasheet" "" (at 93.98 81.28 0)
+      (effects (font (size 1.27 1.27)) hide)
+    )
+    (pin "1")
+    (instances
+      (project "BLDC-Controller"
+        (path "/3f98b8cc-f1be-42b2-9c23-c425b8147bc0/5281a03e-d6ab-4142-84eb-776fec16e050"
+          (reference "#PWR049") (unit 1)
+        )
+        (path "/3f98b8cc-f1be-42b2-9c23-c425b8147bc0/69c4c952-9785-4038-8411-bd74bb4cf876"
+          (reference "#PWR019") (unit 1)
+        )
+      )
+      (project "Honeydew"
+        (path "/534caec7-cf60-4f90-b1ed-42c9d445ef0f/d133c1c6-f35d-4b98-81a0-3607ab1d2de1"
+          (reference "#PWR023") (unit 1)
+        )
+      )

Commit message: Completed initial prototype.
Parts:
- removed U6: TPS62933, Package_TO_SOT_SMD:SOT-583-8, symbol Regulator_Switching:TPS62933
Changed lines of the file:
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@@
 (kicad_sch (version 20230121) (generator eeschema)
   (paper "A4")
-  (junction (at 83.82 58.42) (diameter 0) (color 0 0 0 0)
-  )
-  (wire (pts (xy 83.82 55.88) (xy 83.82 58.42))
-    (stroke (width 0) (type default))
-  )
-  (wire (pts (xy 86.36 60.96) (xy 83.82 60.96))
-    (stroke (width 0) (type default))
-  )
-  (wire (pts (xy 83.82 60.96) (xy 83.82 58.42))
-    (stroke (width 0) (type default))
-  )
-  (wire (pts (xy 93.98 81.28) (xy 93.98 78.74))
-    (stroke (width 0) (type default))
-  )
-  (wire (pts (xy 83.82 58.42) (xy 86.36 58.42))
-    (stroke (width 0) (type default))
-  )
-  (symbol (lib_id "Regulator_Switching:TPS62933") (at 93.98 66.04 0) (unit 1)
-    (in_bom yes) (on_board yes) (dnp no) (fields_autoplaced)
-    (property "Reference" "U6" (at 93.98 51.7357 0)
-      (effects (font (size 1.27 1.27)))
-    )
-    (property "Value" "TPS62933" (at 93.98 54.1599 0)
-      (effects (font (size 1.27 1.27)))
-    )
-    (property "Footprint" "Package_TO_SOT_SMD:SOT-583-8" (at 93.98 91.44 0)
-      (effects (font (size 1.27 1.27)) hide)
-    )
-    (property "Datasheet" "https://www.ti.com/lit/ds/symlink/tps62933.pdf" (at 93.98 88.9 0)
-      (effects (font (size 1.27 1.27)) hide)
-    )
-    (property "Manufacturer no." "" (at 93.98 66.04 0)
-      (effects (font (size 1.27 1.27)) hide)
-    )
-    (pin "1")
-    (pin "2")
-    (pin "3")
-    (pin "4")
-    (pin "5")
-    (pin "6")
-    (pin "7")
-    (pin "8")
-    (instances
-      (project "BLDC-Controller"
-        (path "/3f98b8cc-f1be-42b2-9c23-c425b8147bc0/69c4c952-9785-4038-8411-bd74bb4cf876"
-          (reference "U6") (unit 1)
-        )
-      )
-    )
-  )
-  (symbol (lib_id "power:VCC") (at 83.82 55.88 0) (unit 1)
-    (in_bom yes) (on_board yes) (dnp no) (fields_autoplaced)
-    (property "Reference" "#PWR018" (at 83.82 59.69 0)
-      (effects (font (size 1.27 1.27)) hide)
-    )
-    (property "Value" "VCC" (at 83.82 51.7469 0)
-      (effects (font (size 1.27 1.27)))
-    )
-    (property "Footprint" "" (at 83.82 55.88 0)
-      (effects (font (size 1.27 1.27)) hide)
-    )
-    (property "Datasheet" "" (at 83.82 55.88 0)
-      (effects (font (size 1.27 1.27)) hide)
-    )
-    (pin "1")
-    (instances
-      (project "BLDC-Controller"
-        (path "/3f98b8cc-f1be-42b2-9c23-c425b8147bc0/69c4c952-9785-4038-8411-bd74bb4cf876"
-          (reference "#PWR018") (unit 1)
-        )
-      )
-    )
-  )
-  (symbol (lib_id "power:GND") (at 93.98 81.28 0) (unit 1)
-    (in_bom yes) (on_board yes) (dnp no)
-    (property "Reference" "#PWR049" (at 93.98 87.63 0)
-      (effects (font (size 1.27 1.27)) hide)
-    )
-    (property "Value" "GND" (at 93.98 85.09 0)
-      (effects (font (size 1.27 1.27)) hide)
-    )
-    (property "Footprint" "" (at 93.98 81.28 0)
-      (effects (font (size 1.27 1.27)) hide)
-    )
-    (property "Datasheet" "" (at 93.98 81.28 0)
-      (effects (font (size 1.27 1.27)) hide)
-    )
-    (pin "1")
-    (instances
-      (project "BLDC-Controller"
-        (path "/3f98b8cc-f1be-42b2-9c23-c425b8147bc0/5281a03e-d6ab-4142-84eb-776fec16e050"
-          (reference "#PWR049") (unit 1)
-        )
-        (path "/3f98b8cc-f1be-42b2-9c23-c425b8147bc0/69c4c952-9785-4038-8411-bd74bb4cf876"
-          (reference "#PWR019") (unit 1)
-        )
-      )
-      (project "Honeydew"
-        (path "/534caec7-cf60-4f90-b1ed-42c9d445ef0f/d133c1c6-f35d-4b98-81a0-3607ab1d2de1"
-          (reference "#PWR023") (unit 1)
-        )
-      )
-    )
-  )
 )
