File: PCB/Phase.kicad_sch (KiCad schematic)
At the start: 17 parts, among them Q1 Q_NMOS_GDS, Q2 Q_NMOS_GDS, U1 UCC27211ADRM

Commit message: First draft of schematic done.
Parts:
- removed C2: 10n, Ariamelon-Device:C_0603_1608Metric, symbol Device:C_Small
- removed C4, C5: 4u7, Ariamelon-Device:C_0805_2012Metric, symbol Device:C_Small
- removed L1: L_Small, Ariamelon-Device:L_0603_1608Metric, symbol Device:L_Small
- added C13 (x2): 1000u, Capacitor_THT:CP_Radial_D16.0mm_P7.50mm, symbol Device:C_Polarized_Small
- added D3, D4: 15V, Diode_THT:D_DO-41_SOD81_P7.62mm_Horizontal, symbol Device:D_Zener_Small
- added D5, D6: 400x, Diode_THT:D_DO-41_SOD81_P7.62mm_Horizontal, symbol Device:D_Small
- added R1: 10, Resistor_THT:R_Axial_DIN0207_L6.3mm_D2.5mm_P7.62mm_Horizontal, symbol Device:R_Small
- C1: value 1u -> 10u; footprint Ariamelon-Device:C_0603_1608Metric -> Capacitor_THT:C_Disc_D6.0mm_W2.5mm_P5.00mm
- C2: renamed from C3; footprint Ariamelon-Device:C_0603_1608Metric -> Capacitor_THT:C_Disc_D6.0mm_W2.5mm_P5.00mm
- D1, D2: footprint Ariamelon-Device:D_SOD-323 -> Diode_THT:D_DO-35_SOD27_P7.62mm_Horizontal
- Q1, Q2: value Q_NMOS_GDS -> IRFZ44N; footprint Ariamelon-Package:TO-252-2 -> Package_TO_SOT_THT:TO-220-3_Vertical
- R2: renamed from R3; footprint Ariamelon-Device:R_0603_1608Metric -> Resistor_THT:R_Axial_DIN0207_L6.3mm_D2.5mm_P7.62mm_Horizontal
- R3: renamed from R4; footprint Ariamelon-Device:R_0603_1608Metric -> Resistor_THT:R_Axial_DIN0207_L6.3mm_D2.5mm_P7.62mm_Horizontal
- R4: renamed from R1; footprint Ariamelon-Device:R_0603_1608Metric -> Resistor_THT:R_Axial_DIN0207_L6.3mm_D2.5mm_P7.62mm_Horizontal
- R5: renamed from R2; footprint Ariamelon-Device:R_0603_1608Metric -> Resistor_THT:R_Axial_DIN0207_L6.3mm_D2.5mm_P7.62mm_Horizontal
- R6: renamed from R5; footprint Ariamelon-Device:R_0603_1608Metric -> Resistor_THT:R_Axial_DIN0207_L6.3mm_D2.5mm_P7.62mm_Horizontal
- R7: renamed from R6; footprint Ariamelon-Device:R_0603_1608Metric -> Resistor_THT:R_Axial_DIN0207_L6.3mm_D2.5mm_P7.62mm_Horizontal
- U1: value UCC27211ADRM -> UCC27282
Connections:
- net GNDREF is gone; now on net GND: Q2.3 (S), R7.2
- net GND: now also C13.2, C13.2, D4.2 (A), D6.2 (A)
- net Phase_Out: now also D3.2 (A), D5.2 (A), D6.1 (K)
- net VCC: now also C13.1, C13.1, D5.1 (K)
- net at C1.2, U1.1 (VDD): now also R1.2
- net at Q1.1 (G), R2.2, R4.2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: now also D3.1 (K)
- net at Q2.1 (G), R3.2, R5.2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: now also D4.1 (K)
- new net +12V: R1.1
Other:
- note added: "-3dB point = 1.59kHz"
- note added: "FET gates discharge faster than they charge to avoid cross-conduction"
- note added: "No need for any special circuitry to prevent this"
- note added: "Selected value = 1u (increase if necessary)"
- note added: "UCC27282 has input interlock protection"
- note removed: "= 10 * 49 = 490nF"
- note removed: "Cb > 10 * Qg"
- note removed: "Cboot equations"
- note removed: "Qg = 49nC @ 4.5V"
- note removed: "Selected value = 1u"
- moved on the sheet: C1, C2, D1, D2, Q1, Q2, R2, R3, R4, R5, R6, R7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

Commit message: 28/10/2023 update
Began initial PCB layout.
Parts:
- removed C13: 1000u, Capacitor_THT:CP_Radial_D16.0mm_P7.50mm, symbol Device:C_Polarized_Small
- C1: footprint Capacitor_THT:C_Disc_D6.0mm_W2.5mm_P5.00mm -> Ariamelon-Device:CP_Radial_D5.0mm_P2.54mm; symbol Device:C_Small -> Device:C_Polarized_Small
- C13: footprint Capacitor_THT:CP_Radial_D16.0mm_P7.50mm -> Ariamelon-Device:CP_Radial_D16.0mm_P7.62mm
- C2: value 1u -> 680n; footprint Capacitor_THT:C_Disc_D6.0mm_W2.5mm_P5.00mm -> Ariamelon-Device:C_Rect_L7.0mm_W4.5mm_P5.08mm
- D3, D4, D5, D6: footprint Diode_THT:D_DO-41_SOD81_P7.62mm_Horizontal -> Diode_THT:D_DO-35_SOD27_P7.62mm_Horizontal
- Q1, Q2: value IRFZ44N -> P75NF75
- R1: value 10 -> 1; footprint Resistor_THT:R_Axial_DIN0207_L6.3mm_D2.5mm_P7.62mm_Horizontal -> Resistor_THT:R_Axial_DIN0204_L3.6mm_D1.6mm_P7.62mm_Horizontal
- R2, R3, R4, R5, R6, R7: footprint Resistor_THT:R_Axial_DIN0207_L6.3mm_D2.5mm_P7.62mm_Horizontal -> Resistor_THT:R_Axial_DIN0204_L3.6mm_D1.6mm_P7.62mm_Horizontal
- U1: footprint Ariamelon-Package:SOIC-8_3.9x4.9mm_P1.27mm -> Package_DIP:DIP-8_W7.62mm_Socket
Connections:
- net GND: now also C1.2; no longer C1.1
- net at R1.2, U1.1 (VDD): now also C1.1; no longer C1.2
Other:
- note added: "-3dB point = 15.9kHz"
- note removed: "-3dB point = 1.59kHz"

Commit message: 30/10/2023 update
Completed initial PCB layout.
Parts:
- removed C13: 1000u, Ariamelon-Device:CP_Radial_D16.0mm_P7.62mm, symbol Device:C_Polarized_Small
