File: PCB/BLDC-Controller.kicad_pcb (KiCad board)
At the start: 2 copper layers, 13 parts, among them J1 TC2030-NL, Q1 TPHR8504PL, Q2 TPHR8504PL, Q3 TPHR8504PL, Q4 TPHR8504PL, Q5 TPHR8504PL, Q6 TPHR8504PL, U1 UCC27282, U2 INA180A3, U3 UCC27282, U4 STM32F051K6Ux, U5 UCC27282, U6 TPS62933

Commit message: d
Parts:
- removed J1: TC2030-NL, Connector:Tag-Connect_TC2030-IDC-NL_2x03_P1.27mm_Vertical
- added C1: 1u, Ariamelon-Device:C_0603_1608Metric, F.Cu at (115.5, 84.2)
- added C10: 1u, Ariamelon-Device:C_0603_1608Metric, F.Cu at (115.5, 87.2)
- added C11: 4u7, Ariamelon-Device:C_1206_3216Metric, F.Cu at (169.0, 112.8)
- added C12: 4u7, Ariamelon-Device:C_1206_3216Metric, F.Cu at (169.0, 115.9)
- added C13: 1u, Ariamelon-Device:C_0603_1608Metric, F.Cu at (115.5, 95.4)
- added C14: 100n, Ariamelon-Device:C_0603_1608Metric, F.Cu at (114.1, 95.4)
- added C15: 1n, Ariamelon-Device:C_0603_1608Metric, F.Cu at (114.1, 92.8)
- added C16: 1u, Ariamelon-Device:C_0603_1608Metric, F.Cu at (115.5, 92.8)
- added C17: 4u7, Ariamelon-Device:C_1206_3216Metric, F.Cu at (169.0, 118.5)
- added C18: 4u7, Ariamelon-Device:C_1206_3216Metric, F.Cu at (169.0, 121.5)
- added C19: 4u7, Ariamelon-Device:C_0603_1608Metric, F.Cu at (164.6, 91.4)
- added C2: 100n, Ariamelon-Device:C_0603_1608Metric, F.Cu at (114.1, 84.2)
- added C20: 100n, Ariamelon-Device:C_0603_1608Metric, F.Cu at (164.2, 80.1)
- added C21: 100n, Ariamelon-Device:C_0603_1608Metric, F.Cu at (164.2, 82.0)
- added C22: 4u7, Ariamelon-Device:C_0603_1608Metric, F.Cu at (164.6, 93.7)
- added C23: 10n, Ariamelon-Device:C_0603_1608Metric, F.Cu at (164.2, 83.8)
- added C24: 100p, Ariamelon-Device:C_0603_1608Metric, F.Cu at (164.2, 85.7)
- added C25: 100p, Ariamelon-Device:C_0603_1608Metric, F.Cu at (164.2, 87.5)
- added C26: 100p, Ariamelon-Device:C_0603_1608Metric, F.Cu at (164.2, 89.3)
- added C27: 100p, Ariamelon-Device:C_0603_1608Metric, F.Cu at (166.9, 80.1)
- added C28: 1u, Ariamelon-Device:C_0603_1608Metric, F.Cu at (164.6, 95.9)
- added C3: 1n, Ariamelon-Device:C_0603_1608Metric, F.Cu at (114.1, 81.6)
- added C4: 1u, Ariamelon-Device:C_0603_1608Metric, F.Cu at (115.5, 81.6)
- added C5: 4u7, Ariamelon-Device:C_1206_3216Metric, F.Cu at (169.0, 107.2)
- added C6: 4u7, Ariamelon-Device:C_1206_3216Metric, F.Cu at (169.0, 110.3)
- added C7: 1u, Ariamelon-Device:C_0603_1608Metric, F.Cu at (115.5, 89.8)
- added C8: 100n, Ariamelon-Device:C_0603_1608Metric, F.Cu at (114.1, 89.8)
- added C9: 1n, Ariamelon-Device:C_0603_1608Metric, F.Cu at (114.1, 87.2)
- added D1: 4148, Diode_SMD:D_SOD-123, F.Cu at (118.7, 81.5)
- added D2: 4148, Diode_SMD:D_SOD-123, F.Cu at (118.7, 84.3)
- added D3: 4148, Diode_SMD:D_SOD-123, F.Cu at (118.7, 87.1)
- added D4: 4148, Diode_SMD:D_SOD-123, F.Cu at (118.7, 89.9)
- added D5: 4148, Diode_SMD:D_SOD-123, F.Cu at (118.7, 92.7)
- added D6: 4148, Diode_SMD:D_SOD-123, F.Cu at (118.7, 95.5)
- added R1: 22, Ariamelon-Device:R_0603_1608Metric, F.Cu at (122.4, 82.2)
- added R10: 22, Ariamelon-Device:R_0603_1608Metric, F.Cu at (122.4, 94.8)
- added R11: 10, Ariamelon-Device:R_0603_1608Metric, F.Cu at (122.4, 92.0)
- added R12: 10, Ariamelon-Device:R_0603_1608Metric, F.Cu at (122.4, 96.2)
- added R13: 10k, Ariamelon-Device:R_0402_1005Metric, F.Cu at (166.9, 82.0)
- added R14: 10k, Ariamelon-Device:R_0402_1005Metric, F.Cu at (166.9, 83.8)
- added R15: 10k, Ariamelon-Device:R_0402_1005Metric, F.Cu at (166.9, 85.7)
- added R16: 1k5, Ariamelon-Device:R_0402_1005Metric, F.Cu at (166.9, 87.5)
- added R18: 1k5, Ariamelon-Device:R_0402_1005Metric, F.Cu at (166.9, 89.3)
- added R19: 10k, Ariamelon-Device:R_0402_1005Metric, F.Cu at (169.5, 80.1)
- added R2: 22, Ariamelon-Device:R_0603_1608Metric, F.Cu at (122.4, 83.6)
- added R20: 1k5, Ariamelon-Device:R_0402_1005Metric, F.Cu at (169.5, 82.0)
- added R21: 220, Ariamelon-Device:R_0402_1005Metric, F.Cu at (169.5, 83.8)
- added R3: 10, Ariamelon-Device:R_0603_1608Metric, F.Cu at (122.4, 80.8)
- added R4: 10, Ariamelon-Device:R_0603_1608Metric, F.Cu at (122.4, 85.0)
- added R5: 22, Ariamelon-Device:R_0603_1608Metric, F.Cu at (122.4, 87.8)
- added R6: 22, Ariamelon-Device:R_0603_1608Metric, F.Cu at (122.4, 89.2)
- added R7: 10, Ariamelon-Device:R_0603_1608Metric, F.Cu at (122.4, 86.4)
- added R8: 10, Ariamelon-Device:R_0603_1608Metric, F.Cu at (122.4, 90.6)
- added R9: 22, Ariamelon-Device:R_0603_1608Metric, F.Cu at (122.4, 93.4)
- added Y1: 8M, Crystal:Resonator_SMD_Murata_CSTxExxV-3Pin_3.0x1.1mm, F.Cu at (173.1, 100.0)
- U1, U3: value UCC27282 -> UCC27282DRM; footprint Ariamelon-Package:SOIC-8_3.9x4.9mm_P1.27mm -> Ariamelon-Package:Texas_S-PVSON-N8-1EP_4x4mm_P0.8_EP2.5x3.4mm
- U2: value INA180A3 -> UCC27282DRM; footprint Package_TO_SOT_SMD:SOT-23-5 -> Ariamelon-Package:Texas_S-PVSON-N8-1EP_4x4mm_P0.8_EP2.5x3.4mm
- U5: value UCC27282 -> INA180A3; footprint Ariamelon-Package:SOIC-8_3.9x4.9mm_P1.27mm -> Package_TO_SOT_SMD:SOT-23-5
- moved U5 88.9 mm to (173.4, 93.7)
- moved U6 75.9 mm to (182.7, 112.0)
- moved U4 61.9 mm to (174.5, 87.9)
- moved U3 29.1 mm to (110.8, 93.8), turned to 180 degrees
- moved U1 15.6 mm to (110.8, 82.6), turned to 180 degrees
- moved U2 14.7 mm to (110.8, 88.2), turned to 180 degrees
- moved Q5 1.88 mm to (127.5, 94.1)
- moved Q6 1.70 mm to (135.1, 94.1)
- moved Q3 1.20 mm to (127.5, 88.5)
- moved Q4 0.90 mm to (135.1, 88.5)
- moved Q1 0.81 mm to (127.5, 82.9)
- moved Q2 0.11 mm to (135.1, 82.9)
Connections:
- U2 pad 2: GND -> Net-(U2-HB)
- U2 pad 3: GNDREF -> Net-(D3-K)
- U2 pad 4: GND -> /MCU/Phase_Out_B
- U2 pad 5: +3V3_REF -> /MCU/HI_B
- U3 pad 4: /MCU/Phase_Out_B -> /MCU/Phase_Out_C
- U3 pad 5: /MCU/HI_B -> /MCU/HI_C
- U3 pad 6: /MCU/LI_B -> /MCU/LI_C
- U4 pad 10: V_Sen_B -> V_Sen_A
- U4 pad 11: V_Sen_A -> V_Sen_B
- U4 pad 12: unconnected-(U4-PA6-Pad12) -> V_Sen_A
- U4 pad 2: unconnected-(U4-PF0-Pad2) -> Net-(U4-PF0)
- U4 pad 27: /MCU/PWM_In -> unconnected-(U4-PB4-Pad27)
- U4 pad 3: unconnected-(U4-PF1-Pad3) -> Net-(U4-PF1)
- U4 pad 6: V_Sen_C -> unconnected-(U4-PA0-Pad6)
- U4 pad 7: V_Sen_Com -> unconnected-(U4-PA1-Pad7)
- U4 pad 8: I_Sen -> /MCU/PWM_In
- U4 pad 9: unconnected-(U4-PA3-Pad9) -> I_Sen
- U5 pad 2: Net-(U5-HB) -> GND
- U5 pad 3: Net-(D5-K) (its old number) -> GNDREF
- U5 pad 4: /MCU/Phase_Out_C -> GND
- U5 pad 5: /MCU/HI_C -> +3V3_REF

Commit message: f
Parts:
- C1, C10, C13, C16, C4, C7, Q1, Q3, Q5: moved to B.Cu
- C11, C12, C17, C18, C5, C6: footprint Ariamelon-Device:C_1206_3216Metric -> Ariamelon-Device:C_0805_2012Metric; moved to B.Cu
- C14, C2, C8: value 100n -> 10n; moved to B.Cu
- C15, C3, C9: value 1n -> 10n; moved to B.Cu
- C22: value 4u7 -> 1u
- U1, U2, U3: footprint Ariamelon-Package:Texas_S-PVSON-N8-1EP_4x4mm_P0.8_EP2.5x3.4mm -> Ariamelon-Package:SOIC-8_3.9x4.9mm_P1.27mm; moved to B.Cu
- moved C12 54.2 mm to (122.2, 88.5)
- moved C18 54.2 mm to (122.2, 94.1)
- moved C6 54.2 mm to (122.2, 82.9)
- moved C11 53.6 mm to (122.2, 86.7)
- moved C17 53.6 mm to (122.2, 92.3)
- moved C5 53.6 mm to (122.2, 81.1)
- moved U6 28.5 mm to (160.2, 94.6)
- moved Y1 24.4 mm to (151.5, 88.6)
- moved R19 23.2 mm to (147.6, 87.6)
- moved R20 23.2 mm to (147.6, 89.5)
- moved R21 23.1 mm to (147.6, 76.5)
- moved C19 20.3 mm to (150.6, 76.7)
- moved R13 19.6 mm to (147.6, 78.4)
- moved R14 19.6 mm to (147.6, 80.2)
- moved R15 19.6 mm to (147.6, 82.1)
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Connections:
- net /MCU/USART_RX renamed /MCU/USART1_RX
- net /MCU/USART_TX renamed /MCU/USART1_TX
- C14 pad 1: GND -> Net-(U3-VDD)
- C14 pad 2: Net-(U3-VDD) -> GND
- C2 pad 1: GND -> Net-(U1-VDD)
- C2 pad 2: Net-(U1-VDD) -> GND
- C8 pad 1: GND -> Net-(U2-VDD)
- C8 pad 2: Net-(U2-VDD) -> GND
- U4 pad 10: V_Sen_A -> V_Sen_B
- U4 pad 11: V_Sen_B -> V_Sen_A
- U4 pad 12: V_Sen_A -> unconnected-(U4-PA6-Pad12)
- U4 pad 27: unconnected-(U4-PB4-Pad27) -> /MCU/PWM_In
- U4 pad 7: unconnected-(U4-PA1-Pad7) -> I_Sen
- U4 pad 8: /MCU/PWM_In -> V_Sen_In
- U4 pad 9: I_Sen -> V_Sen_A
Routing:
- net Net-(D6-K): track 0.00 -> 5.16 mm
- net Net-(D1-K): track 0.00 -> 5.16 mm
- net Net-(D4-K): track 0.00 -> 5.16 mm
- net Net-(D3-K): track 0.00 -> 5.16 mm
- net Net-(D5-K): track 0.00 -> 5.16 mm
- net Net-(D2-K): track 0.00 -> 5.16 mm
- net Net-(D6-A): track 0.00 -> 1.53 mm
- net Net-(D5-A): track 0.00 -> 1.53 mm
- net Net-(D4-A): track 0.00 -> 1.53 mm
- net Net-(D3-A): track 0.00 -> 1.53 mm
- net Net-(D2-A): track 0.00 -> 1.53 mm
- net Net-(D1-A): track 0.00 -> 1.53 mm
- net Net-(Q6-G): track 0.00 -> 1.40 mm
- net Net-(Q5-G): track 0.00 -> 1.40 mm
- net Net-(Q2-G): track 0.00 -> 1.40 mm
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- added copper zone on B.Cu, net GNDREF
- added copper zone on F.Cu, net GNDREF
- added copper zone on B.Cu, net VCC

Commit message: f
Parts:
- added R11: 100k, Ariamelon-Device:R_0603_1608Metric, F.Cu at (152.1, 115.9)
- added R12: 100k, Ariamelon-Device:R_0603_1608Metric, F.Cu at (166.6, 116.6)
- added R26: 100k, Ariamelon-Device:R_0603_1608Metric, F.Cu at (152.1, 125.1)
- added R27: 100k, Ariamelon-Device:R_0603_1608Metric, F.Cu at (166.6, 125.8)
- added R5: 100k, Ariamelon-Device:R_0603_1608Metric, F.Cu at (152.1, 106.7)
- added R6: 100k, Ariamelon-Device:R_0603_1608Metric, F.Cu at (166.6, 107.4)
- Q1, Q3, Q5: value TPHR8504PL -> Q_NMOS_GDS; footprint Ariamelon-Package:SOP-8-Advance_5.0x6.0mm_P1.27mm -> Package_TO_SOT_SMD:TO-252-2; moved to F.Cu
- Q2, Q4, Q6: value TPHR8504PL -> Q_NMOS_GDS; footprint Ariamelon-Package:SOP-8-Advance_5.0x6.0mm_P1.27mm -> Package_TO_SOT_SMD:TO-252-2
- moved Q6 42.9 mm to (158.8, 123.5), turned to 180 degrees
- moved Q4 40.5 mm to (158.8, 114.3), turned to 180 degrees
- moved Q2 38.3 mm to (158.8, 105.1), turned to 180 degrees
- moved Q5 34.1 mm to (144.9, 123.5)
- moved Q3 31.1 mm to (144.9, 114.3)
- moved Q1 28.1 mm to (144.9, 105.1)
- renumbered R8 to R10, R9 to R22, R10 to R23, R11 to R24, R12 to R25, R5 to R7, R6 to R8, R7 to R9
Connections:
- Q1 pad 1: /MCU/Phase_Out_A -> Net-(Q1-G)
- Q1 pad 2: /MCU/Phase_Out_A -> VCC
- Q2 pad 1: GNDREF -> Net-(Q2-G)
- Q2 pad 2: GNDREF -> /MCU/Phase_Out_A
- Q3 pad 1: /MCU/Phase_Out_B -> Net-(Q3-G)
- Q3 pad 2: /MCU/Phase_Out_B -> VCC
- Q4 pad 1: GNDREF -> Net-(Q4-G)
- Q4 pad 2: GNDREF -> /MCU/Phase_Out_B
- Q5 pad 1: /MCU/Phase_Out_C -> Net-(Q5-G)
- Q5 pad 2: /MCU/Phase_Out_C -> VCC
- Q6 pad 1: GNDREF -> Net-(Q6-G)
- Q6 pad 2: GNDREF -> /MCU/Phase_Out_C
Routing:
- added copper zone on F.Cu, net /MCU/Phase_Out_A
- added copper zone on F.Cu, net /MCU/Phase_Out_B
- added copper zone on F.Cu, net /MCU/Phase_Out_C

Commit message: f
Parts:
- removed the C15 at (115.7, 95.4)
- removed the C3 at (115.7, 84.2)
- removed the C9 at (115.7, 89.8)
- removed the R22 at (116.5, 93.4)
- removed R23: 22, Ariamelon-Device:R_0603_1608Metric
- removed the R24 at (116.5, 92.0)
- removed the R25 at (116.5, 96.2)
- added L1: L_Small, Ariamelon-Device:L_0603_1608Metric, B.Cu at (153.3, 107.6)
- added L2: L_Small, Ariamelon-Device:L_0603_1608Metric, B.Cu at (178.8, 99.0)
- added L3: L_Small, Ariamelon-Device:L_0603_1608Metric, B.Cu at (173.3, 94.7)
- added R13: 10, Ariamelon-Device:R_0603_1608Metric, B.Cu at (180.1, 105.6)
- added R14: 10, Ariamelon-Device:R_0603_1608Metric, B.Cu at (180.1, 107.8)
- added R15: 22, Ariamelon-Device:R_0603_1608Metric, B.Cu at (180.1, 110.1)
- added R16: 22, Ariamelon-Device:R_0603_1608Metric, B.Cu at (180.1, 112.3)
- C16: renamed from C19; moved to B.Cu
- C17: renamed from C20; moved to B.Cu
- C18: renamed from C21; moved to B.Cu
- C19: renamed from C22; moved to B.Cu
- C20: renamed from C23; moved to B.Cu
- C21: renamed from C24; moved to B.Cu
- C22: renamed from C26; moved to B.Cu
- C23: renamed from C25; moved to B.Cu
- C24: renamed from C28; moved to B.Cu
- C25: renamed from C27; moved to B.Cu
- D1, D2, D3, D4, D5, D6: footprint Diode_SMD:D_SOD-123 -> Ariamelon-Device:D_SOD-323; moved to B.Cu
- Q1, Q2, Q3, Q4, Q5, Q6: footprint Package_TO_SOT_SMD:TO-252-2 -> Ariamelon-Package:TO-252-2
- R1, R2, R7, R8: value 22 -> 10; moved to B.Cu
- R10, R3, R4, R9: value 10 -> 22; moved to B.Cu
- R19: renamed from R21; moved to B.Cu
- R20: renamed from R13; moved to B.Cu
- R21: renamed from R14; moved to B.Cu
- R22: renamed from R15; moved to B.Cu
- R24: renamed from R16; moved to B.Cu
- R25: renamed from R18; moved to B.Cu
- R26: renamed from R19; moved to B.Cu
- R27: renamed from R20; moved to B.Cu
- U1, U2, U3: value UCC27282DRM -> UCC27211ADRM
- U4: value STM32F051K6Ux -> STM32F051K6Tx; footprint Package_DFN_QFN:QFN-32-1EP_5x5mm_P0.5mm_EP3.45x3.45mm -> Package_QFP:LQFP-32_7x7mm_P0.8mm; moved to B.Cu
- U5, Y1: moved to B.Cu
- moved R9 82.4 mm to (191.3, 121.1), turned to 180 degrees
- moved R10 81.6 mm to (191.3, 123.3), turned to 180 degrees
- moved R8 80.4 mm to (191.3, 118.8), turned to 180 degrees
- moved R7 80.1 mm to (191.3, 116.6), turned to 180 degrees
- moved D4 79.8 mm to (186.7, 120.5), turned to 180 degrees
- moved D3 79.8 mm to (186.7, 117.2), turned to 180 degrees
- moved D6 64.1 mm to (175.4, 109.5), turned to 180 degrees
- moved D2 57.7 mm to (166.0, 107.0), turned to 90 degrees
- moved U3 56.6 mm to (161.2, 120.9), turned to 0 degrees
- moved R4 55.9 mm to (167.7, 107.4), turned to 90 degrees
- moved U2 55.8 mm to (161.2, 113.5), turned to 0 degrees
- moved U1 55.0 mm to (161.2, 106.1), turned to 0 degrees
- moved R2 54.5 mm to (166.8, 104.6)
- moved C12 50.7 mm to (156.7, 122.7)
- moved D5 50.4 mm to (155.7, 118.9), turned to 180 degrees
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- renumbered C12 to C10, C13 to C11, C14 to C12, C16 to C13, C17 to C14, C18 to C15, C4 to C3, C5 to C4, C6 to C5, C7 to C6, C8 to C7, C10 to C8, C11 to C9, R26 to R17, R27 to R18
Connections:
- R1 pad 1: Net-(D1-K) -> Net-(D1-A)
- R10 pad 1: Net-(D4-A) -> Net-(D4-K)
- R2 pad 1: Net-(D2-K) -> Net-(D2-A)
- R3 pad 1: Net-(D1-A) -> Net-(D1-K)
- R4 pad 1: Net-(D2-A) -> Net-(D2-K)
- R7 pad 1: Net-(D3-K) -> Net-(D3-A)
- R8 pad 1: Net-(D4-K) -> Net-(D4-A)
- R9 pad 1: Net-(D3-A) -> Net-(D3-K)
- U4 pad 13: /MCU/LI_C -> /MCU/LI_A
- U4 pad 15: /MCU/LI_A -> /MCU/LI_C
- U4 pad 16: unconnected-(U4-PB2-Pad16) -> GND
- U4 pad 18: /MCU/HI_C -> /MCU/HI_A
- U4 pad 20: /MCU/HI_A -> /MCU/HI_C
- U4 pad 32: unconnected-(U4-PB8-Pad32) -> GND
Routing:
- net Net-(Q2-G): track 1.40 -> 6.95 mm, vias 0 -> 1
- net Net-(D6-K): track 5.16 -> 0.00 mm
- net Net-(D1-K): track 5.16 -> 0.00 mm
- net Net-(D4-K): track 5.16 -> 0.00 mm
- net Net-(D3-K): track 5.16 -> 0.00 mm
- net Net-(D5-K): track 5.16 -> 0.00 mm
- net Net-(U1-VDD): track 0.00 -> 2.84 mm
- net Net-(Q1-G): track 1.40 -> 3.46 mm
- net Net-(D6-A): track 1.53 -> 0.00 mm
- net Net-(D5-A): track 1.53 -> 0.00 mm
- net Net-(D4-A): track 1.53 -> 0.00 mm
- net Net-(D3-A): track 1.53 -> 0.00 mm
- net Net-(D1-A): track 1.53 -> 0.00 mm
- net Net-(Q6-G): track 1.40 -> 0.00 mm
- net Net-(Q4-G): track 1.40 -> 0.00 mm
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- added copper zone on F.Cu, net VCC

Commit message: First draft of schematic done.
Parts:
- removed L1, L2, L3: L_Small, Ariamelon-Device:L_0603_1608Metric
- added C26: 1n, Capacitor_THT:C_Disc_D6.0mm_W2.5mm_P5.00mm, F.Cu at (134.1, 60.8)
- added C27: 22p, Capacitor_THT:C_Disc_D5.0mm_W2.5mm_P2.50mm, F.Cu at (137.9, 93.0)
- added C28: 22p, Capacitor_THT:C_Disc_D5.0mm_W2.5mm_P2.50mm, F.Cu at (137.9, 97.1)
- added D10: 15V, Diode_THT:D_DO-41_SOD81_P7.62mm_Horizontal, F.Cu at (133.4, 107.6)
- added D11: 400x, Diode_THT:D_DO-41_SOD81_P7.62mm_Horizontal, F.Cu at (133.4, 111.8)
- added D12: 400x, Diode_THT:D_DO-41_SOD81_P7.62mm_Horizontal, F.Cu at (133.4, 116.1)
- added D13: 4148, Diode_THT:D_DO-35_SOD27_P7.62mm_Horizontal, F.Cu at (175.3, 120.0)
- added D14: 4148, Diode_THT:D_DO-35_SOD27_P7.62mm_Horizontal, F.Cu at (175.3, 123.5)
- added D15: 15V, Diode_THT:D_DO-41_SOD81_P7.62mm_Horizontal, F.Cu at (175.6, 103.3)
- added D16: 15V, Diode_THT:D_DO-41_SOD81_P7.62mm_Horizontal, F.Cu at (175.6, 107.6)
- added D17: 400x, Diode_THT:D_DO-41_SOD81_P7.62mm_Horizontal, F.Cu at (175.6, 111.8)
- added D18: 400x, Diode_THT:D_DO-41_SOD81_P7.62mm_Horizontal, F.Cu at (175.6, 116.1)
- added D19: 400x, Diode_THT:D_DO-41_SOD81_P7.62mm_Horizontal, F.Cu at (144.3, 69.0)
- added D20: 400x, Diode_THT:D_DO-41_SOD81_P7.62mm_Horizontal, F.Cu at (144.3, 73.2)
- added D21: 400x, Diode_THT:D_DO-41_SOD81_P7.62mm_Horizontal, F.Cu at (144.3, 77.5)
- added D7: 4148, Diode_THT:D_DO-35_SOD27_P7.62mm_Horizontal, F.Cu at (133.1, 120.0)
- added D8: 4148, Diode_THT:D_DO-35_SOD27_P7.62mm_Horizontal, F.Cu at (133.1, 123.5)
- added D9: 15V, Diode_THT:D_DO-41_SOD81_P7.62mm_Horizontal, F.Cu at (133.4, 103.3)
- added J1: Prog, Connector_PinSocket_2.54mm:PinSocket_1x04_P2.54mm_Vertical, F.Cu at (115.8, 78.0)
- added J2: Receiver, Connector_PinSocket_2.54mm:PinSocket_1x03_P2.54mm_Vertical, F.Cu at (120.4, 78.0)
- added J3: ICSP, Connector_PinSocket_2.54mm:PinSocket_2x03_P2.54mm_Vertical, F.Cu at (118.4, 90.2)
- added R23: 560, Resistor_THT:R_Axial_DIN0207_L6.3mm_D2.5mm_P7.62mm_Horizontal, F.Cu at (104.3, 44.5)
- added R28: 47k, Resistor_THT:R_Axial_DIN0207_L6.3mm_D2.5mm_P7.62mm_Horizontal, F.Cu at (104.3, 64.8)
- added R29: 47k, Resistor_THT:R_Axial_DIN0207_L6.3mm_D2.5mm_P7.62mm_Horizontal, F.Cu at (104.3, 68.8)
- added R30: 47k, Resistor_THT:R_Axial_DIN0207_L6.3mm_D2.5mm_P7.62mm_Horizontal, F.Cu at (104.3, 72.9)
- added R31: 4k7, Resistor_THT:R_Axial_DIN0207_L6.3mm_D2.5mm_P7.62mm_Horizontal, F.Cu at (104.3, 77.0)
- added R32: 4k7, Resistor_THT:R_Axial_DIN0207_L6.3mm_D2.5mm_P7.62mm_Horizontal, F.Cu at (104.3, 81.0)
- added R33: 4k7, Resistor_THT:R_Axial_DIN0207_L6.3mm_D2.5mm_P7.62mm_Horizontal, F.Cu at (104.3, 85.0)
- added R34: 47k, Resistor_THT:R_Axial_DIN0207_L6.3mm_D2.5mm_P7.62mm_Horizontal, F.Cu at (104.3, 89.1)
- added R35: 47k, Resistor_THT:R_Axial_DIN0207_L6.3mm_D2.5mm_P7.62mm_Horizontal, F.Cu at (104.3, 93.2)
- added R36: 47k, Resistor_THT:R_Axial_DIN0207_L6.3mm_D2.5mm_P7.62mm_Horizontal, F.Cu at (104.3, 97.2)
- added SW1: RST, Button_Switch_THT:SW_PUSH_6mm, F.Cu at (142.7, 40.5)
- added SW2: Speed+, Button_Switch_THT:SW_PUSH_6mm, F.Cu at (142.7, 49.0)
- added SW3: Speed-, Button_Switch_THT:SW_PUSH_6mm, F.Cu at (142.7, 57.6)
- C1, C19: value 1u -> 10u; footprint Ariamelon-Device:C_0603_1608Metric -> Capacitor_THT:C_Disc_D6.0mm_W2.5mm_P5.00mm; moved to F.Cu
- C10, C14: value 4u7 -> 1u; footprint Ariamelon-Device:C_0805_2012Metric -> Capacitor_THT:C_Disc_D6.0mm_W2.5mm_P5.00mm; moved to F.Cu
- C11, C13, C3, C8: value 1u -> 1000u; footprint Ariamelon-Device:C_0603_1608Metric -> Capacitor_THT:CP_Radial_D16.0mm_P7.50mm; moved to F.Cu
- C12, C7: value 10n -> 1000u; footprint Ariamelon-Device:C_0603_1608Metric -> Capacitor_THT:CP_Radial_D16.0mm_P7.50mm; moved to F.Cu
- C15, C5, C9: value 4u7 -> 10u; footprint Ariamelon-Device:C_0805_2012Metric -> Capacitor_THT:C_Disc_D6.0mm_W2.5mm_P5.00mm; moved to F.Cu
- C16: value 4u7 -> 10u; footprint Ariamelon-Device:C_0603_1608Metric -> Capacitor_THT:C_Disc_D6.0mm_W2.5mm_P5.00mm; moved to F.Cu
- C17, C18: value 100n -> 10u; footprint Ariamelon-Device:C_0603_1608Metric -> Capacitor_THT:C_Disc_D6.0mm_W2.5mm_P5.00mm; moved to F.Cu
- C2: value 10n -> 1u; footprint Ariamelon-Device:C_0603_1608Metric -> Capacitor_THT:C_Disc_D6.0mm_W2.5mm_P5.00mm; moved to F.Cu
- C20: value 10n -> 100n; footprint Ariamelon-Device:C_0603_1608Metric -> Capacitor_THT:C_Disc_D6.0mm_W2.5mm_P5.00mm; moved to F.Cu
- C21, C22: value 100p -> 100n; footprint Ariamelon-Device:C_0603_1608Metric -> Capacitor_THT:C_Disc_D6.0mm_W2.5mm_P5.00mm; moved to F.Cu
- C23: value 100p -> 1n; footprint Ariamelon-Device:C_0603_1608Metric -> Capacitor_THT:C_Disc_D6.0mm_W2.5mm_P5.00mm; moved to F.Cu
- C24: value 1u -> 1n; footprint Ariamelon-Device:C_0603_1608Metric -> Capacitor_THT:C_Disc_D6.0mm_W2.5mm_P5.00mm; moved to F.Cu
- C25: value 100p -> 22p; footprint Ariamelon-Device:C_0603_1608Metric -> Capacitor_THT:C_Disc_D6.0mm_W2.5mm_P5.00mm; moved to F.Cu
- C4: value 4u7 -> 1000u; footprint Ariamelon-Device:C_0805_2012Metric -> Capacitor_THT:CP_Radial_D16.0mm_P7.50mm; moved to F.Cu
- C6: footprint Ariamelon-Device:C_0603_1608Metric -> Capacitor_THT:C_Disc_D6.0mm_W2.5mm_P5.00mm; moved to F.Cu
- D1, D2: footprint Ariamelon-Device:D_SOD-323 -> Diode_THT:D_DO-35_SOD27_P7.62mm_Horizontal; moved to F.Cu
- D3, D4: value 4148 -> 15V; footprint Ariamelon-Device:D_SOD-323 -> Diode_THT:D_DO-41_SOD81_P7.62mm_Horizontal; moved to F.Cu
- D5, D6: value 4148 -> 400x; footprint Ariamelon-Device:D_SOD-323 -> Diode_THT:D_DO-41_SOD81_P7.62mm_Horizontal; moved to F.Cu
- Q1, Q2, Q3, Q4, Q5, Q6: value Q_NMOS_GDS -> IRFZ44N; footprint Ariamelon-Package:TO-252-2 -> Package_TO_SOT_THT:TO-220-3_Vertical
- R1, R10, R16, R3, R8, R9: footprint Ariamelon-Device:R_0603_1608Metric -> Resistor_THT:R_Axial_DIN0207_L6.3mm_D2.5mm_P7.62mm_Horizontal; moved to F.Cu
- R11, R12, R18, R5: value 100k -> 10; footprint Ariamelon-Device:R_0603_1608Metric -> Resistor_THT:R_Axial_DIN0207_L6.3mm_D2.5mm_P7.62mm_Horizontal
- R13, R14, R7: value 10 -> 100k; footprint Ariamelon-Device:R_0603_1608Metric -> Resistor_THT:R_Axial_DIN0207_L6.3mm_D2.5mm_P7.62mm_Horizontal; moved to F.Cu
- R15, R4: value 22 -> 10; footprint Ariamelon-Device:R_0603_1608Metric -> Resistor_THT:R_Axial_DIN0207_L6.3mm_D2.5mm_P7.62mm_Horizontal; moved to F.Cu
- R17: value 100k -> 22; footprint Ariamelon-Device:R_0603_1608Metric -> Resistor_THT:R_Axial_DIN0207_L6.3mm_D2.5mm_P7.62mm_Horizontal
- R19: value 220 -> 10; footprint Ariamelon-Device:R_0402_1005Metric -> Resistor_THT:R_Axial_DIN0207_L6.3mm_D2.5mm_P7.62mm_Horizontal; moved to F.Cu
- R2: value 10 -> 22; footprint Ariamelon-Device:R_0603_1608Metric -> Resistor_THT:R_Axial_DIN0207_L6.3mm_D2.5mm_P7.62mm_Horizontal; moved to F.Cu
- R20, R21: value 10k -> 100k; footprint Ariamelon-Device:R_0402_1005Metric -> Resistor_THT:R_Axial_DIN0207_L6.3mm_D2.5mm_P7.62mm_Horizontal; moved to F.Cu
- R22: value 10k -> 4k7; footprint Ariamelon-Device:R_0402_1005Metric -> Resistor_THT:R_Axial_DIN0207_L6.3mm_D2.5mm_P7.62mm_Horizontal; moved to F.Cu
- R24: value 1k5 -> 10; footprint Ariamelon-Device:R_0402_1005Metric -> Resistor_THT:R_Axial_DIN0207_L6.3mm_D2.5mm_P7.62mm_Horizontal; moved to F.Cu
- R25, R27: value 1k5 -> 10k; footprint Ariamelon-Device:R_0402_1005Metric -> Resistor_THT:R_Axial_DIN0207_L6.3mm_D2.5mm_P7.62mm_Horizontal; moved to F.Cu
- R26: footprint Ariamelon-Device:R_0402_1005Metric -> Resistor_THT:R_Axial_DIN0207_L6.3mm_D2.5mm_P7.62mm_Horizontal; moved to F.Cu
- R6: footprint Ariamelon-Device:R_0603_1608Metric -> Resistor_THT:R_Axial_DIN0207_L6.3mm_D2.5mm_P7.62mm_Horizontal
- U1, U2, U3: moved to F.Cu
- U4: value STM32F051K6Tx -> ATmega328P-P; footprint Package_QFP:LQFP-32_7x7mm_P0.8mm -> Package_DIP:DIP-28_W7.62mm; moved to F.Cu
- U5: value INA180A3 -> LM317; footprint Package_TO_SOT_SMD:SOT-23-5 -> Package_TO_SOT_THT:TO-220-3_Vertical; moved to F.Cu
- U6: value TPS62933 -> LM7805; footprint Package_TO_SOT_SMD:SOT-583-8 -> Package_TO_SOT_THT:TO-220-3_Vertical
- Y1: value 8M -> 16M; footprint Crystal:Resonator_SMD_Murata_CSTxExxV-3Pin_3.0x1.1mm -> Crystal:Crystal_HC49-U_Vertical; moved to F.Cu
- moved D3 76.6 mm to (186.4, 40.6), turned to 0 degrees
- moved D5 76.3 mm to (186.4, 49.1), turned to 0 degrees
- moved D4 75.7 mm to (186.4, 44.9), turned to 0 degrees
- moved R22 72.9 mm to (104.3, 40.5), turned to 0 degrees
- moved C10 71.6 mm to (176.1, 135.7)
- moved R8 70.7 mm to (122.3, 103.2), turned to 0 degrees
- moved R9 70.3 mm to (122.3, 107.3), turned to 0 degrees
- moved U4 70.3 mm to (115.1, 40.5)
- moved C9 70.1 mm to (176.1, 131.6)
- moved R10 70.0 mm to (122.3, 111.3), turned to 0 degrees
- moved R1 69.5 mm to (175.3, 40.5), turned to 0 degrees
- moved R24 69.5 mm to (104.3, 48.6), turned to 0 degrees
- moved R25 68.4 mm to (104.3, 52.6), turned to 0 degrees
- moved R26 67.3 mm to (104.3, 56.7), turned to 0 degrees
- moved R27 66.4 mm to (104.3, 60.8), turned to 0 degrees
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Connections:
- C10 pad 1: GNDREF -> /MCU/Phase_Out_C
- C10 pad 2: VCC -> Net-(U3-HB)
- C11 pad 1: GND -> VCC
- C11 pad 2: Net-(U3-VDD) -> GND
- C12 pad 1: Net-(U3-VDD) -> VCC
- C13 pad 1: /MCU/Phase_Out_C -> VCC
- C13 pad 2: Net-(U3-HB) -> GND
- C14 pad 1: GNDREF -> VCC
- C14 pad 2: VCC -> GND
- C15 pad 1: GNDREF -> GND
- C15 pad 2: VCC -> +5V
- C16 pad 2: +3V3 -> +12V
- C17 pad 2: +3V3 -> +12V
- C18 pad 2: +3V3 -> Net-(D21-K)
- C19 pad 2: +3V3_REF -> +5V
- C2 pad 1: Net-(U1-VDD) -> /MCU/Phase_Out_A
- C2 pad 2: GND -> Net-(U1-HB)
- C20 pad 1: GND -> RST
- C20 pad 2: +3V3_REF -> GND
- C21 pad 1: GND -> Speed+
- C21 pad 2: V_Sen_A -> GND
- C22 pad 1: GND -> Speed-
- C22 pad 2: I_Sen -> GND
- C23 pad 2: V_Sen_B -> V_Sen_A
- C24 pad 2: +3V3_REF -> V_Sen_B
- C25 pad 2: V_Sen_A -> PWM_In
- C3 pad 1: /MCU/Phase_Out_A -> VCC
- C3 pad 2: Net-(U1-HB) -> GND
- C4 pad 1: GNDREF -> VCC
- C4 pad 2: VCC -> GND
- C5 pad 1: GNDREF -> GND
- C5 pad 2: VCC -> Net-(U2-VDD)
- C6 pad 1: GND -> /MCU/Phase_Out_B
- C6 pad 2: Net-(U2-VDD) -> Net-(U2-HB)
- C7 pad 1: Net-(U2-VDD) -> VCC
- C8 pad 1: /MCU/Phase_Out_B -> VCC
- C8 pad 2: Net-(U2-HB) -> GND
- C9 pad 1: GNDREF -> GND
- C9 pad 2: VCC -> Net-(U3-VDD)
- D3 pad 2: Net-(D3-A) -> /MCU/Phase_Out_A
- D4 pad 2: Net-(D4-A) -> GND
- D5 pad 1: Net-(D5-K) -> VCC
- D5 pad 2: Net-(D5-A) -> /MCU/Phase_Out_A
- D6 pad 1: Net-(D6-K) -> /MCU/Phase_Out_A
- D6 pad 2: Net-(D6-A) -> GND
- Q1 pad 1: Net-(Q1-G) -> Net-(D3-K)
- Q2 pad 1: Net-(Q2-G) -> Net-(D4-K)
- Q2 pad 3: GNDREF -> GND
- Q3 pad 1: Net-(Q3-G) -> Net-(D9-K)
- Q4 pad 1: Net-(Q4-G) -> Net-(D10-K)
- Q4 pad 3: GNDREF -> GND
- Q5 pad 1: Net-(Q5-G) -> Net-(D15-K)
- Q6 pad 1: Net-(Q6-G) -> Net-(D16-K)
- Q6 pad 3: GNDREF -> GND
- R1 pad 1: Net-(D1-A) -> +12V
- R1 pad 2: Net-(Q1-G) -> Net-(U1-VDD)
- R10 pad 1: Net-(D4-K) -> Net-(D8-K)
- R10 pad 2: Net-(Q4-G) -> Net-(D10-K)
- R11 pad 1: Net-(Q3-G) -> Net-(D7-A)
- R11 pad 2: /MCU/Phase_Out_B -> Net-(D9-K)
- R12 pad 1: Net-(Q4-G) -> Net-(D8-A)
- R12 pad 2: GNDREF -> Net-(D10-K)
- R13 pad 1: Net-(D5-A) -> Net-(D9-K)
- R13 pad 2: Net-(Q5-G) -> /MCU/Phase_Out_B
- R14 pad 1: Net-(D6-A) -> Net-(D10-K)
- R14 pad 2: Net-(Q6-G) -> GND
- R15 pad 1: Net-(D5-K) -> +12V
- R15 pad 2: Net-(Q5-G) -> Net-(U3-VDD)
- R16 pad 1: Net-(D6-K) -> Net-(D13-K)
- R16 pad 2: Net-(Q6-G) -> Net-(D15-K)
- R17 pad 1: Net-(Q5-G) -> Net-(D14-K)
- R17 pad 2: /MCU/Phase_Out_C -> Net-(D16-K)
- R18 pad 1: Net-(Q6-G) -> Net-(D13-A)
- R18 pad 2: GNDREF -> Net-(D15-K)
- R19 pad 1: Net-(U4-PF1) -> Net-(D14-A)
- R19 pad 2: Net-(R19-Pad2) -> Net-(D16-K)
- R2 pad 1: Net-(D2-A) -> Net-(D1-K)
- R2 pad 2: Net-(Q2-G) -> Net-(D3-K)
- R20 pad 1: V_Sen_A -> Net-(D15-K)
- R20 pad 2: /MCU/Phase_Out_A -> /MCU/Phase_Out_C
- R21 pad 1: V_Sen_B -> Net-(D16-K)
- R21 pad 2: /MCU/Phase_Out_B -> GND
- R22 pad 1: V_Sen_A -> GND
- R22 pad 2: /MCU/Phase_Out_C -> Net-(U5-ADJ)
- R24 pad 1: GND -> +12V
- R24 pad 2: V_Sen_A -> Net-(D21-K)
- R25 pad 1: GND -> +5V
- R25 pad 2: V_Sen_B -> RST
- R26 pad 1: I_Sen -> +5V
- R26 pad 2: Net-(R26-Pad2) -> Speed+
- R27 pad 1: GND -> +5V
- R27 pad 2: V_Sen_A -> Speed-
- R3 pad 1: Net-(D1-K) -> Net-(D2-K)
- R3 pad 2: Net-(Q1-G) -> Net-(D4-K)
- R4 pad 1: Net-(D2-K) -> Net-(D1-A)
- R4 pad 2: Net-(Q2-G) -> Net-(D3-K)
- R5 pad 1: Net-(Q1-G) -> Net-(D2-A)
- R5 pad 2: /MCU/Phase_Out_A -> Net-(D4-K)
- R6 pad 1: Net-(Q2-G) -> Net-(D3-K)
- R6 pad 2: GNDREF -> /MCU/Phase_Out_A
- R7 pad 1: Net-(D3-A) -> Net-(D4-K)
- R7 pad 2: Net-(Q3-G) -> GND
- R8 pad 1: Net-(D4-A) -> +12V
- R8 pad 2: Net-(Q4-G) -> Net-(U2-VDD)
- R9 pad 1: Net-(D3-K) -> Net-(D7-K)
- R9 pad 2: Net-(Q3-G) -> Net-(D9-K)
- U1 pad 5: /MCU/HI_A -> RX
- U2 pad 3: Net-(D3-K) -> Net-(D7-K)
- U2 pad 5: /MCU/HI_B -> TX
- U2 pad 8: Net-(D4-K) -> Net-(D8-K)
- U3 pad 3: Net-(D5-K) -> Net-(D13-K)
- U3 pad 8: Net-(D6-K) -> Net-(D14-K)
- U4 pad 1: +3V3 -> RST
- U4 pad 10: V_Sen_B -> XTAL2
- U4 pad 11: V_Sen_A -> unconnected-(U4-PD5-Pad11)
- U4 pad 12: unconnected-(U4-PA6-Pad12) -> V_Sen_COM
- U4 pad 13: /MCU/LI_A -> unconnected-(U4-PD7-Pad13)
- U4 pad 14: /MCU/LI_B -> PWM_In
- U4 pad 15: /MCU/LI_C -> Speed+
- U4 pad 16: GND -> Speed-
- U4 pad 17: +3V3 -> MOSI
- U4 pad 18: /MCU/HI_A -> MISO
- U4 pad 19: /MCU/HI_B -> SCK
- U4 pad 2: Net-(U4-PF0) -> RX
- U4 pad 20: /MCU/HI_C -> +5V
- U4 pad 21: unconnected-(U4-PA11-Pad21) -> +5V
- U4 pad 22: unconnected-(U4-PA12-Pad22) -> GND
- U4 pad 23: SWD -> V_Sen_A
- U4 pad 24: SWC -> V_Sen_B
- U4 pad 25: unconnected-(U4-PA15-Pad25) -> V_Sen_A
- U4 pad 26: unconnected-(U4-PB3-Pad26) -> /MCU/LI_A
- U4 pad 27: /MCU/PWM_In -> /MCU/LI_B
- U4 pad 28: unconnected-(U4-PB5-Pad28) -> /MCU/LI_C
- U4 pad 3: Net-(U4-PF1) -> TX
- U4 pad 4: RST -> /MCU/HI_C
- U4 pad 5: +3V3_REF -> unconnected-(U4-PD3-Pad5)
- U4 pad 7: I_Sen -> +5V
- U4 pad 8: V_Sen_In -> GND
- U4 pad 9: V_Sen_A -> XTAL1
- U5 pad 1: Net-(R26-Pad2) -> Net-(U5-ADJ)
- U5 pad 2: GND -> +12V
- U5 pad 3: GNDREF -> VCC
- U6 pad 1: unconnected-(U6-RT-Pad1) -> Net-(D21-K)
- U6 pad 2: VCC -> GND
- U6 pad 3: VCC -> +5V
- Y1 pad 1: Net-(U4-PF0) -> XTAL1
- Y1 pad 2: GND -> XTAL2
Routing:
- net Net-(Q2-G): track 6.95 -> 0.00 mm, vias 1 -> 0
- net Net-(D2-K): track 3.89 -> 0.00 mm
- net Net-(Q1-G): track 3.46 -> 0.00 mm
- net Net-(U1-VDD): track 2.84 -> 0.00 mm
- net Net-(Q5-G): track 2.16 -> 0.00 mm
- net Net-(Q3-G): track 2.16 -> 0.00 mm
- net Net-(U2-VDD): track 1.40 -> 0.00 mm
- net Net-(D2-A): track 1.20 -> 0.00 mm
- net GNDREF: track 1.00 -> 0.00 mm, vias 36 -> 0
- removed copper zone on F.Cu, net /MCU/Phase_Out_A
- removed copper zone on F.Cu, net /MCU/Phase_Out_B
- removed copper zone on F.Cu, net /MCU/Phase_Out_C
- removed copper zone on B.Cu, net GNDREF
- removed copper zone on F.Cu, net GNDREF
- removed copper zone on B.Cu, net VCC
- removed copper zone on F.Cu, net VCC
