File: PCB/BLDC-Controller.kicad_pcb (KiCad board)
At the start: 2 copper layers, 114.3 x 76.5 mm, 95 parts, among them J1 Prog, J2 Receiver, J3 Bat_In, J4 Mot_Con, J5 Mot_Con, J6 Mot_Con, Q1 P75NF75, Q2 P75NF75, Q3 P75NF75, Q4 P75NF75, Q5 P75NF75, Q6 P75NF75, SW1 RST, SW2 Speed+, SW3 Speed-, U1 UCC27282, U2 UCC27282, U3 UCC27282, U4 ATmega328P-P, U5 LM317, U6 LM7805, Y1 16M

Commit message: V2 started
Parts:
- removed A1: Art, Ariamelon-Logo:Ariamelon_Logo_Large_Mask
- removed D10, D15, D16, D4, D9: 15V, Diode_THT:D_DO-35_SOD27_P7.62mm_Horizontal
- removed D11, D12, D17, D18, D19, D20, D21, D5, D6: 400x, Diode_THT:D_DO-35_SOD27_P7.62mm_Horizontal
- removed D13, D14, D7, D8: 4148, Diode_THT:D_DO-35_SOD27_P7.62mm_Horizontal
- removed the J1 at (130.0, 91.7)
- removed R19: 10, Resistor_THT:R_Axial_DIN0204_L3.6mm_D1.6mm_P7.62mm_Horizontal
- removed R20, R21: 100k, Resistor_THT:R_Axial_DIN0204_L3.6mm_D1.6mm_P7.62mm_Horizontal
- removed R22, R29, R30, R31: 4k7, Resistor_THT:R_Axial_DIN0204_L3.6mm_D1.6mm_P7.62mm_Horizontal
- removed R23: 560, Resistor_THT:R_Axial_DIN0204_L3.6mm_D1.6mm_P7.62mm_Horizontal
- removed R24: 1, Resistor_THT:R_Axial_DIN0204_L3.6mm_D1.6mm_P7.62mm_Horizontal
- removed R25: 10k, Resistor_THT:R_Axial_DIN0204_L3.6mm_D1.6mm_P7.62mm_Horizontal
- removed R26, R27, R28, R32, R33, R34: 47k, Resistor_THT:R_Axial_DIN0204_L3.6mm_D1.6mm_P7.62mm_Horizontal
- added C21: 10u, Ariamelon-Device:C_0805_2012Metric, F.Cu at (36.6, 61.4)
- added C22: 22p, Ariamelon-Device:C_0603_1608Metric, F.Cu at (46.9, 18.6)
- added J10: Receiver, Connector_PinHeader_2.54mm:PinHeader_1x03_P2.54mm_Vertical, F.Cu at (71.5, 70.2)
- added J4: Mot_Con, TestPoint:TestPoint_Pad_4.0x4.0mm, B.Cu at (74.0, 29.9)
- added J7: Bat+, Ariamelon-HolePad:MountingHole_3.2mm_M3_Pad, F.Cu at (171.7, 66.5)
- added J8: Bat-, Ariamelon-HolePad:MountingHole_3.2mm_M3_Pad, F.Cu at (171.7, 73.7)
- added J9: Prog, Connector_PinHeader_2.54mm:PinHeader_1x06_P2.54mm_Vertical, F.Cu at (58.2, 91.7)
- added R1: 10, Ariamelon-Device:R_0603_1608Metric, F.Cu at (63.8, 42.1)
- added R15: 33k, Ariamelon-Device:R_0603_1608Metric, F.Cu at (55.2, 63.2)
- added R8: 33k, Ariamelon-Device:R_0603_1608Metric, F.Cu at (72.3, 38.9)
- C1, C14, C18, C19, C3, C5: footprint Ariamelon-Device:CP_Radial_D5.0mm_P2.54mm -> Ariamelon-Device:C_0805_2012Metric
- C10, C12: value 10u -> 100n; footprint Ariamelon-Device:CP_Radial_D5.0mm_P2.54mm -> Ariamelon-Device:C_0603_1608Metric
- C11: value 10u -> 1000u; footprint Ariamelon-Device:CP_Radial_D5.0mm_P2.54mm -> Ariamelon-Device:CP_Radial_D16.0mm_P7.62mm
- C13: value 22p -> 1000u; footprint Ariamelon-Device:C_Disc_D5.0mm_W2.5mm_P2.54mm -> Ariamelon-Device:CP_Radial_D16.0mm_P7.62mm
- C15: footprint Ariamelon-Device:C_Disc_D5.0mm_W2.5mm_P2.54mm -> Ariamelon-Device:C_0603_1608Metric
- C16: value 470u -> 22p; footprint Capacitor_THT:CP_Radial_D10.0mm_P5.00mm -> Ariamelon-Device:C_0603_1608Metric
- C17: value 100n -> 10u; footprint Ariamelon-Device:C_Disc_D6.0mm_W2.5mm_P5.08mm -> Ariamelon-Device:C_0805_2012Metric
- C2, C4, C6: value 680n -> 2u2; footprint Ariamelon-Device:C_Rect_L7.0mm_W4.5mm_P5.08mm -> Ariamelon-Device:C_0805_2012Metric
- C20: value 22p -> 100n; footprint Ariamelon-Device:C_Disc_D5.0mm_W2.5mm_P2.54mm -> Ariamelon-Device:C_0603_1608Metric
- C7: value 1000u -> 10u; footprint Ariamelon-Device:CP_Radial_D16.0mm_P7.62mm -> Ariamelon-Device:C_0805_2012Metric
- C8: value 1000u -> 100n; footprint Ariamelon-Device:CP_Radial_D16.0mm_P7.62mm -> Ariamelon-Device:C_0603_1608Metric
- D1, D2: value 4148 -> 400x; footprint Diode_THT:D_DO-35_SOD27_P7.62mm_Horizontal -> Diode_SMD:D_SOD-123F
- D3: value 15V -> 400x; footprint Diode_THT:D_DO-35_SOD27_P7.62mm_Horizontal -> Diode_SMD:D_SOD-123F
- J1: renamed from J4; footprint Ariamelon-HolePad:MountingHole_3.2mm_M3_Pad -> TestPoint:TestPoint_Pad_4.0x4.0mm
- J2: value Receiver -> Mot_Con; footprint Connector_PinHeader_2.54mm:PinHeader_1x03_P2.54mm_Vertical -> TestPoint:TestPoint_Pad_4.0x4.0mm; moved to B.Cu
- J3: value Bat_In -> Mot_Con; footprint Connector_AMASS:AMASS_XT60-M_1x02_P7.20mm_Vertical -> TestPoint:TestPoint_Pad_4.0x4.0mm
- J5: footprint Ariamelon-HolePad:MountingHole_3.2mm_M3_Pad -> TestPoint:TestPoint_Pad_4.0x4.0mm
- J6: footprint Ariamelon-HolePad:MountingHole_3.2mm_M3_Pad -> TestPoint:TestPoint_Pad_4.0x4.0mm; moved to B.Cu
- Q1, Q2, Q3, Q4, Q5, Q6: footprint Package_TO_SOT_THT:TO-220-3_Vertical -> Ariamelon-Package:TO-252-2; moved to B.Cu
- R10, R3: value 22 -> 33k; footprint Resistor_THT:R_Axial_DIN0204_L3.6mm_D1.6mm_P7.62mm_Horizontal -> Ariamelon-Device:R_0603_1608Metric
- R11, R12: footprint Resistor_THT:R_Axial_DIN0204_L3.6mm_D1.6mm_P7.62mm_Horizontal -> Ariamelon-Device:R_0603_1608Metric
- R13: value 100k -> 33k; footprint Resistor_THT:R_Axial_DIN0204_L3.6mm_D1.6mm_P7.62mm_Horizontal -> Ariamelon-Device:R_0603_1608Metric
- R14: value 100k -> 10k; footprint Resistor_THT:R_Axial_DIN0204_L3.6mm_D1.6mm_P7.62mm_Horizontal -> Ariamelon-Device:R_0603_1608Metric
- R16, R9: value 22 -> 10k; footprint Resistor_THT:R_Axial_DIN0204_L3.6mm_D1.6mm_P7.62mm_Horizontal -> Ariamelon-Device:R_0603_1608Metric
- R17: value 22 -> 560; footprint Resistor_THT:R_Axial_DIN0204_L3.6mm_D1.6mm_P7.62mm_Horizontal -> Ariamelon-Device:R_0603_1608Metric
- R18, R4: value 10 -> 10k; footprint Resistor_THT:R_Axial_DIN0204_L3.6mm_D1.6mm_P7.62mm_Horizontal -> Ariamelon-Device:R_0603_1608Metric
- R2: value 22 -> 10; footprint Resistor_THT:R_Axial_DIN0204_L3.6mm_D1.6mm_P7.62mm_Horizontal -> Ariamelon-Device:R_0603_1608Metric
- R5: value 10 -> 33k; footprint Resistor_THT:R_Axial_DIN0204_L3.6mm_D1.6mm_P7.62mm_Horizontal -> Ariamelon-Device:R_0603_1608Metric
- R6, R7: value 100k -> 10; footprint Resistor_THT:R_Axial_DIN0204_L3.6mm_D1.6mm_P7.62mm_Horizontal -> Ariamelon-Device:R_0603_1608Metric
- U1, U2, U3: footprint Package_DIP:DIP-8_W7.62mm_Socket -> Package_SO:SOIC-8_3.9x4.9mm_P1.27mm
- U4: value ATmega328P-P -> ATmega328P-A; footprint Package_DIP:DIP-28_W7.62mm_Socket -> Package_QFP:TQFP-32_7x7mm_P0.8mm
- U6: value LM7805 -> L78L05; footprint Package_TO_SOT_THT:TO-220-3_Vertical -> Package_TO_SOT_SMD:SOT-89-3
- Y1: footprint Crystal:Crystal_HC49-4H_Vertical -> Crystal:Crystal_SMD_3225-4Pin_3.2x2.5mm
- moved C20 132.3 mm to (46.9, 16.3)
- moved C13 128.5 mm to (22.0, 59.1)
- moved SW1 113.7 mm to (36.6, 17.2), turned to 0 degrees
- moved R17 110.9 mm to (46.9, 23.1), turned to 0 degrees
- moved J2 110.8 mm to (66.8, 29.9), turned to 0 degrees
- moved R18 105.0 mm to (46.9, 25.3), turned to 0 degrees
- moved SW2 100.2 mm to (36.6, 25.8), turned to 0 degrees
- moved C17 97.5 mm to (36.6, 53.5), turned to 0 degrees
- moved R16 96.7 mm to (46.9, 20.8), turned to 0 degrees
- moved SW3 92.0 mm to (36.6, 34.3), turned to 0 degrees
- moved C12 82.4 mm to (65.8, 62.7), turned to -90 degrees
- moved C15 79.2 mm to (82.3, 60.2), turned to -90 degrees
- moved C19 76.1 mm to (36.6, 58.8), turned to 0 degrees
- moved Q6 74.1 mm to (81.2, 38.8), turned to -90 degrees
- moved Y1 73.8 mm to (79.9, 60.1), turned to 90 degrees
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Connections:
- C13 pad 1: GND -> VCC
- C13 pad 2: XTAL1 -> GND
- C14 pad 1: Net-(D20-A) -> VCC
- C15 pad 2: XTAL2 -> XTAL1
- C16 pad 1: +12V -> GND
- C16 pad 2: GND -> XTAL2
- C17 pad 1: RST -> Net-(D2-A)
- C18 pad 1: Net-(D21-K) -> +12V
- C19 pad 1: +5V -> +12V
- C2 pad 1: /MCU/Phase_Out_A -> /Phase A/Phase_Out
- C20 pad 1: GND -> RST
- C20 pad 2: PWM_In -> GND
- C4 pad 1: /MCU/Phase_Out_B -> /Phase B/Phase_Out
- C6 pad 1: /MCU/Phase_Out_C -> /Phase C/Phase_Out
- C7 pad 1: VCC -> +5V
- C8 pad 1: VCC -> +5V
- D1 pad 1: Net-(D1-K) -> VCC
- D1 pad 2: Net-(D1-A) -> +12V
- D2 pad 1: Net-(D2-K) -> +12V
- D3 pad 1: Net-(D3-K) -> +12V
- D3 pad 2: /MCU/Phase_Out_A -> +5V
- J1 pad 1: /MCU/Phase_Out_A -> /Phase A/Phase_Out
- J2 pad 1: PWM_In -> /Phase A/Phase_Out
- J3 pad 1: GND -> /Phase B/Phase_Out
- J5 pad 1: /MCU/Phase_Out_B -> /Phase C/Phase_Out
- J6 pad 1: /MCU/Phase_Out_C -> /Phase C/Phase_Out
- Q1 pad 1: Net-(D3-K) -> Net-(Q1-G)
- Q1 pad 3: /MCU/Phase_Out_A -> /Phase A/Phase_Out
- Q2 pad 1: Net-(D4-K) -> Net-(Q2-G)
- Q2 pad 2: /MCU/Phase_Out_A -> /Phase A/Phase_Out
- Q3 pad 1: Net-(D9-K) -> Net-(Q3-G)
- Q3 pad 3: /MCU/Phase_Out_B -> /Phase B/Phase_Out
- Q4 pad 1: Net-(D10-K) -> Net-(Q4-G)
- Q4 pad 2: /MCU/Phase_Out_B -> /Phase B/Phase_Out
- Q5 pad 1: Net-(D15-K) -> Net-(Q5-G)
- Q5 pad 3: /MCU/Phase_Out_C -> /Phase C/Phase_Out
- Q6 pad 1: Net-(D16-K) -> Net-(Q6-G)
- Q6 pad 2: /MCU/Phase_Out_C -> /Phase C/Phase_Out
- R10 pad 1: Net-(D8-K) -> /MCU/V_Sen_B
- R10 pad 2: Net-(D10-K) -> /MCU/V_Sen_COM
- R11 pad 1: Net-(D7-A) -> Net-(Q5-G)
- R11 pad 2: Net-(D9-K) -> Net-(U3-HO)
- R12 pad 1: Net-(D8-A) -> Net-(Q6-G)
- R12 pad 2: Net-(D10-K) -> Net-(U3-LO)
- R13 pad 1: Net-(D9-K) -> /MCU/V_Sen_C
- R13 pad 2: /MCU/Phase_Out_B -> /Phase C/Phase_Out
- R14 pad 1: Net-(D10-K) -> GND
- R14 pad 2: GND -> /MCU/V_Sen_C
- R16 pad 1: Net-(D13-K) -> GND
- R16 pad 2: Net-(D15-K) -> Net-(D2-A)
- R17 pad 1: Net-(D14-K) -> +12V
- R17 pad 2: Net-(D16-K) -> Net-(D2-A)
- R18 pad 1: Net-(D13-A) -> +5V
- R18 pad 2: Net-(D15-K) -> RST
- R2 pad 1: Net-(D1-K) -> Net-(Q2-G)
- R2 pad 2: Net-(D3-K) -> Net-(U1-LO)
- R3 pad 1: Net-(D2-K) -> /MCU/V_Sen_A
- R3 pad 2: Net-(D4-K) -> /Phase A/Phase_Out
- R4 pad 1: Net-(D1-A) -> GND
- R4 pad 2: Net-(D3-K) -> /MCU/V_Sen_A
- R5 pad 1: Net-(D2-A) -> /MCU/V_Sen_A
- R5 pad 2: Net-(D4-K) -> /MCU/V_Sen_COM
- R6 pad 1: Net-(D3-K) -> Net-(Q3-G)
- R6 pad 2: /MCU/Phase_Out_A -> Net-(U2-HO)
- R7 pad 1: Net-(D4-K) -> Net-(Q4-G)
- R7 pad 2: GND -> Net-(U2-LO)
- R9 pad 1: Net-(D7-K) -> GND
- R9 pad 2: Net-(D9-K) -> /MCU/V_Sen_B
- U1 pad 3: Net-(D1-K) -> Net-(U1-HO)
- U1 pad 4: /MCU/Phase_Out_A -> /Phase A/Phase_Out
- U1 pad 8: Net-(D2-K) -> Net-(U1-LO)
- U2 pad 3: Net-(D7-K) -> Net-(U2-HO)
- U2 pad 4: /MCU/Phase_Out_B -> /Phase B/Phase_Out
- U2 pad 8: Net-(D8-K) -> Net-(U2-LO)
- U3 pad 3: Net-(D13-K) -> Net-(U3-HO)
- U3 pad 4: /MCU/Phase_Out_C -> /Phase C/Phase_Out
- U3 pad 8: Net-(D14-K) -> Net-(U3-LO)
- U4 pad 1: RST -> Speed-
- U4 pad 10: XTAL2 -> /MCU/V_Sen_COM
- U4 pad 12: V_Sen_COM -> unconnected-(U4-PB0-Pad12)
- U4 pad 13: unconnected-(U4-PD7-Pad13) -> /MCU/HI_C
- U4 pad 14: PWM_In -> /MCU/HI_B
- U4 pad 15: /MCU/HI_C -> /MCU/HI_A
- U4 pad 16: /MCU/HI_B -> unconnected-(U4-PB4-Pad16)
- U4 pad 17: /MCU/HI_A -> PWM_In
- U4 pad 18: unconnected-(U4-PB4-Pad18) -> +5V
- U4 pad 2: RX -> Speed+
- U4 pad 21: +5V -> GND
- U4 pad 22: GND -> unconnected-(U4-ADC7-Pad22)
- U4 pad 26: V_Sen_C -> /MCU/V_Sen_C
- U4 pad 27: V_Sen_B -> /MCU/V_Sen_B
- U4 pad 28: V_Sen_A -> /MCU/V_Sen_A
- U4 pad 3: TX -> GND
- U4 pad 4: Speed- -> +5V
- U4 pad 5: Speed+ -> GND
- U4 pad 6: unconnected-(U4-PD4-Pad6) -> +5V
- U4 pad 7: +5V -> XTAL1
- U4 pad 8: GND -> XTAL2
- U4 pad 9: XTAL1 -> unconnected-(U4-PD5-Pad9)
- U5 pad 1: Net-(D20-A) -> Net-(D2-A)
- U6 pad 1: Net-(D21-K) -> +5V
- U6 pad 3: +5V -> +12V
- Y1 pad 2: XTAL2 -> GND
Routing:
- net GND: track 238.8 -> 11.5 mm, vias 0 -> 24
- net +12V: track 160.8 -> 5.78 mm
- net +5V: track 105.4 -> 12.9 mm
- net /MCU/HI_A: track 71.2 -> 15.7 mm, vias 1 -> 2
- net V_Sen_C: track 50.0 -> 0.00 mm, vias 1 -> 0
- net V_Sen_A: track 41.9 -> 0.00 mm
- net /MCU/Phase_Out_A: track 41.1 -> 0.00 mm
- net /MCU/Phase_Out_C: track 41.1 -> 0.00 mm
- net /MCU/Phase_Out_B: track 41.0 -> 0.00 mm
- net V_Sen_COM: track 36.9 -> 0.00 mm, vias 1 -> 0
- net Speed+: track 36.3 -> 0.00 mm
- net /MCU/HI_B: track 42.5 -> 10.4 mm, vias 1 -> 2
- net /MCU/LI_A: track 53.6 -> 23.4 mm
- net /MCU/V_Sen_A: track 0.00 -> 28.3 mm, vias 0 -> 1
- net VCC: track 27.2 -> 0.00 mm
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- added copper zone on B.Cu, net /Phase A/Phase_Out
- added copper zone on B.Cu, net /Phase B/Phase_Out
- added copper zone on B.Cu, net /Phase C/Phase_Out
- removed copper zone on B.Cu, net /MCU/Phase_Out_A
- removed copper zone on B.Cu, net /MCU/Phase_Out_B
- removed copper zone on B.Cu, net /MCU/Phase_Out_C
Other:
- board size 114.3 x 76.5 mm -> 24 x 44.2 mm
- board text removed: "0V"
- board text removed: "400x"
- board text removed: "5V"
- board text removed: "BLDC Motor Controller V1.0"
- board text removed: "IN"
- board text removed: "RX"
- board text removed: "TX"

Commit message: f
Parts:
- removed C11, C13, C9: 1000u, Ariamelon-Device:CP_Radial_D16.0mm_P7.62mm
- removed C14, C17, C18, C19, C21, C7: 10u, Ariamelon-Device:C_0805_2012Metric
- removed C20: 100n, Ariamelon-Device:C_0603_1608Metric
- removed C22: 22p, Ariamelon-Device:C_0603_1608Metric
- removed D1, D2, D3: 400x, Diode_SMD:D_SOD-123F
- removed R16, R18: 10k, Ariamelon-Device:R_0603_1608Metric
- removed R17: 560, Ariamelon-Device:R_0603_1608Metric
- removed SW1: RST, Button_Switch_THT:SW_PUSH_6mm
- removed SW2: Speed+, Button_Switch_THT:SW_PUSH_6mm
- removed SW3: Speed-, Button_Switch_THT:SW_PUSH_6mm
- removed U5: LM317, Package_TO_SOT_THT:TO-220-3_Vertical
- removed U6: L78L05, Package_TO_SOT_SMD:SOT-89-3
- moved C12 8.22 mm to (58.9, 67.0), turned to 0 degrees
- moved C16 2.44 mm to (82.0, 58.0), turned to 135 degrees
- moved C10 1.84 mm to (78.0, 65.6)
- moved C8 1.84 mm to (78.0, 63.0)
- moved C15 1.62 mm to (81.7, 61.7), turned to -135 degrees
- moved J10 1.00 mm to (71.5, 71.2)
- moved U4 0.50 mm to (71.6, 63.4)
- moved Y1 0.14 mm to (80.0, 60.0), turned to 45 degrees
Routing:
- net /MCU/LI_C: track 32.7 -> 6.19 mm
- net /MCU/LI_B: track 27.1 -> 6.19 mm
- net /MCU/LI_A: track 23.4 -> 6.19 mm
- net /MCU/HI_C: track 16.1 -> 3.42 mm, vias 2 -> 1
- net /MCU/HI_A: track 15.7 -> 3.42 mm, vias 2 -> 1
- net /MCU/V_Sen_A: track 28.3 -> 17.5 mm, vias 1 -> 0
- net +5V: track 12.9 -> 4.53 mm
- net /MCU/HI_B: track 10.4 -> 3.42 mm, vias 2 -> 1
- net GND: track 11.5 -> 5.45 mm
- net /MCU/V_Sen_C: track 16.7 -> 19.1 mm, vias 1 -> 0
- net XTAL1: track 7.14 -> 4.96 mm
- net XTAL2: track 4.94 -> 6.66 mm
- net /MCU/V_Sen_B: track 16.6 -> 15.2 mm, vias 1 -> 0
Other:
- board size 24 x 44.2 mm -> 24 x 45.2 mm

Commit message: k
Parts:
- moved R14 2.83 mm to (81.9, 39.0), turned to 90 degrees
- moved R9 2.05 mm to (73.7, 39.0), turned to 90 degrees
- moved C6 1.57 mm to (80.5, 41.2)
- moved R11 1.57 mm to (79.6, 42.8)
- moved R12 1.57 mm to (82.6, 51.8)
- moved U3 1.57 mm to (81.1, 47.3)
- moved R4 1.55 mm to (65.5, 39.0), turned to 90 degrees
- moved C5 1.49 mm to (83.0, 41.8)
- moved Q2 1.02 mm to (65.8, 39.0)
- moved Q6 1.02 mm to (82.2, 39.0)
- moved R13 1.00 mm to (80.5, 39.0), turned to -90 degrees
- moved R3 1.00 mm to (64.1, 39.0), turned to -90 degrees
- moved J1 1.00 mm to (65.8, 29.9)
- moved J2 1.00 mm to (65.8, 29.9)
- moved J5 1.00 mm to (82.2, 29.9)
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Routing:
- net /MCU/V_Sen_C: track 19.1 -> 9.87 mm
- net /MCU/LI_C: track 6.19 -> 0.00 mm
- net /MCU/LI_B: track 6.19 -> 0.00 mm
- net /MCU/LI_A: track 6.19 -> 0.00 mm
- net /MCU/V_Sen_B: track 15.2 -> 10.4 mm
- net /MCU/HI_C: track 3.42 -> 0.00 mm, vias 1 -> 0
- net /MCU/HI_B: track 3.42 -> 0.00 mm, vias 1 -> 0
- net /MCU/HI_A: track 3.42 -> 0.00 mm, vias 1 -> 0
- net /Phase C/Phase_Out: track 6.04 -> 9.31 mm, vias 16 -> 17
- net /Phase A/Phase_Out: track 6.04 -> 9.21 mm, vias 16 -> 17
- net /Phase B/Phase_Out: track 6.04 -> 9.20 mm, vias 16 -> 17
- net Net-(Q4-G): track 21.7 -> 23.4 mm
- net Net-(Q2-G): track 21.7 -> 23.3 mm
- net Net-(Q6-G): track 21.7 -> 23.3 mm
- net GND: vias 24 -> 48
Other:
- board size 24 x 45.2 mm -> 26 x 45 mm
