File: PCB/BLDC-Controller.kicad_sch (KiCad schematic)
At the start: 0 parts

Commit message: f
Other:
- added sheet PSU (PSU.kicad_sch)
- sheet MCU ports: added Phase_Out_A, Phase_Out_B, Phase_Out_C; removed I_Sen_A, I_Sen_B, I_Sen_C, V_Sen_A, V_Sen_B, V_Sen_C, V_Sen_In
- sheet Phase A ports: added none; removed I_Sen, V_Sen
- sheet Phase B ports: added none; removed I_Sen, V_Sen
- sheet Phase C ports: added none; removed I_Sen, V_Sen
Changed lines of the file:
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@@
-    (stroke (width 0) (type default))
-  )
-  (wire (pts (xy 170.18 116.84) (xy 180.34 116.84))
-    (stroke (width 0) (type default))
-  )
-  (wire (pts (xy 170.18 68.58) (xy 180.34 68.58))
-    (stroke (width 0) (type default))
-  )
-  (wire (pts (xy 170.18 109.22) (xy 180.34 109.22))
     (stroke (width 0) (type default))
   )
@@
     (stroke (width 0) (type default))
   )
+  (wire (pts (xy 170.18 111.76) (xy 180.34 111.76))
+    (stroke (width 0) (type default))
+  )
+  (wire (pts (xy 170.18 104.14) (xy 180.34 104.14))
+    (stroke (width 0) (type default))
+  )
   (wire (pts (xy 170.18 60.96) (xy 180.34 60.96))
     (stroke (width 0) (type default))
   )
-  (wire (pts (xy 170.18 111.76) (xy 180.34 111.76))
+  (wire (pts (xy 170.18 88.9) (xy 180.34 88.9))
     (stroke (width 0) (type default))
   )
-  (wire (pts (xy 170.18 86.36) (xy 180.34 86.36))
-    (stroke (width 0) (type default))
-  )
-  (wire (pts (xy 170.18 93.98) (xy 180.34 93.98))
-    (stroke (width 0) (type default))
-  )
-  (wire (pts (xy 170.18 91.44) (xy 180.34 91.44))
+  (wire (pts (xy 170.18 106.68) (xy 180.34 106.68))
     (stroke (width 0) (type default))
   )
@@
     (stroke (width 0) (type default))
   )
-  (wire (pts (xy 170.18 119.38) (xy 180.34 119.38))
+  (wire (pts (xy 170.18 81.28) (xy 180.34 81.28))
     (stroke (width 0) (type default))
   )
@@
     (effects (font (size 1.27 1.27)) (justify left bottom))
   )
-  (sheet (at 180.34 81.28) (size 25.4 15.24) (fields_autoplaced)
+  (sheet (at 180.34 78.74) (size 25.4 12.7) (fields_autoplaced)
     (stroke (width 0.1524) (type solid))
     (fill (color 0 0 0 0.0000))
-    (property "Sheetname" "Phase B" (at 180.34 80.5684 0)
+    (property "Sheetname" "Phase B" (at 180.34 78.0284 0)
       (effects (font (size 1.27 1.27)) (justify left bottom))
     )
-    (property "Sheetfile" "Phase.kicad_sch" (at 180.34 97.1046 0)
+    (property "Sheetfile" "Phase.kicad_sch" (at 180.34 92.0246 0)
       (effects (font (size 1.27 1.27)) (justify left top))
     )
-    (pin "V_Sen" output (at 180.34 91.44 180)
+    (pin "Phase_Out" output (at 180.34 88.9 180)
       (effects (font (size 1.27 1.27)) (justify left))
     )
-    (pin "Phase_Out" output (at 205.74 88.9 0)
-      (effects (font (size 1.27 1.27)) (justify right))
-    )
-    (pin "I_Sen" output (at 180.34 93.98 180)
+    (pin "HI" input (at 180.34 81.28 180)
       (effects (font (size 1.27 1.27)) (justify left))
     )
-    (pin "HI" input (at 180.34 83.82 180)
-      (effects (font (size 1.27 1.27)) (justify left))
-    )
-    (pin "LI" input (at 180.34 86.36 180)
+    (pin "LI" input (at 180.34 83.82 180)
       (effects (font (size 1.27 1.27)) (justify left))
     )
@@
     )
   )
-  (sheet (at 180.34 106.68) (size 25.4 15.24) (fields_autoplaced)
+  (sheet (at 180.34 101.6) (size 25.4 12.7) (fields_autoplaced)
     (stroke (width 0.1524) (type solid))
     (fill (color 0 0 0 0.0000))
-    (property "Sheetname" "Phase C" (at 180.34 105.9684 0)
+    (property "Sheetname" "Phase C" (at 180.34 100.8884 0)
       (effects (font (size 1.27 1.27)) (justify left bottom))
     )
-    (property "Sheetfile" "Phase.kicad_sch" (at 180.34 122.5046 0)
+    (property "Sheetfile" "Phase.kicad_sch" (at 180.34 114.8846 0)
       (effects (font (size 1.27 1.27)) (justify left top))
     )
-    (pin "V_Sen" output (at 180.34 116.84 180)
+    (pin "Phase_Out" output (at 180.34 111.76 180)
       (effects (font (size 1.27 1.27)) (justify left))
     )
-    (pin "Phase_Out" output (at 205.74 114.3 0)
-      (effects (font (size 1.27 1.27)) (justify right))
-    )
-    (pin "I_Sen" output (at 180.34 119.38 180)
+    (pin "HI" input (at 180.34 104.14 180)
       (effects (font (size 1.27 1.27)) (justify left))
     )
-    (pin "HI" input (at 180.34 109.22 180)
-      (effects (font (size 1.27 1.27)) (justify left))
-    )
-    (pin "LI" input (at 180.34 111.76 180)
+    (pin "LI" input (at 180.34 106.68 180)
       (effects (font (size 1.27 1.27)) (justify left))
     )
@@
     )
   )
-  (sheet (at 119.38 55.88) (size 50.8 66.04) (fields_autoplaced)
+  (sheet (at 119.38 55.88) (size 50.8 58.42) (fields_autoplaced)
     (stroke (width 0.1524) (type solid))
     (fill (color 0 0 0 0.0000))
@@
       (effects (font (size 1.27 1.27)) (justify left bottom))
     )
-    (property "Sheetfile" "MCU.kicad_sch" (at 119.38 122.5046 0)
+    (property "Sheetfile" "MCU.kicad_sch" (at 119.38 114.8846 0)
       (effects (font (size 1.27 1.27)) (justify left top))
     )
-    (pin "V_Sen_C" input (at 170.18 116.84 0)
-      (effects (font (size 1.27 1.27)) (justify right))
-    )
-    (pin "V_Sen_B" input (at 170.18 91.44 0)
-      (effects (font (size 1.27 1.27)) (justify right))
-    )
-    (pin "V_Sen_A" input (at 170.18 66.04 0)
-      (effects (font (size 1.27 1.27)) (justify right))
-    )
-    (pin "V_Sen_In" input (at 119.38 58.42 180)
-      (effects (font (size 1.27 1.27)) (justify left))
-    )
-    (pin "LI_B" output (at 170.18 86.36 0)
+    (pin "LI_B" output (at 170.18 83.82 0)
       (effects (font (size 1.27 1.27)) (justify right))
     )
@@
       (effects (font (size 1.27 1.27)) (justify right))
     )
-    (pin "HI_B" output (at 170.18 83.82 0)
+    (pin "HI_B" output (at 170.18 81.28 0)
       (effects (font (size 1.27 1.27)) (justify right))
     )
-    (pin "HI_C" output (at 170.18 109.22 0)
+    (pin "HI_C" output (at 170.18 104.14 0)
       (effects (font (size 1.27 1.27)) (justify right))
     )
-    (pin "LI_C" output (at 170.18 111.76 0)
+    (pin "LI_C" output (at 170.18 106.68 0)
       (effects (font (size 1.27 1.27)) (justify right))
     )
-    (pin "I_Sen_A" input (at 170.18 68.58 0)
+    (pin "Phase_Out_C" input (at 170.18 111.76 0)
       (effects (font (size 1.27 1.27)) (justify right))
     )
-    (pin "I_Sen_B" input (at 170.18 93.98 0)
+    (pin "Phase_Out_B" input (at 170.18 88.9 0)
       (effects (font (size 1.27 1.27)) (justify right))
     )
-    (pin "I_Sen_C" input (at 170.18 119.38 0)
+    (pin "Phase_Out_A" input (at 170.18 66.04 0)
       (effects (font (size 1.27 1.27)) (justify right))
     )
@@
     )
   )
-  (sheet (at 180.34 55.88) (size 25.4 15.24) (fields_autoplaced)
+  (sheet (at 180.34 55.88) (size 25.4 12.7) (fields_autoplaced)
     (stroke (width 0.1524) (type solid))
     (fill (color 0 0 0 0.0000))
@@
       (effects (font (size 1.27 1.27)) (justify left bottom))
     )
-    (property "Sheetfile" "Phase.kicad_sch" (at 180.34 71.7046 0)
+    (property "Sheetfile" "Phase.kicad_sch" (at 180.34 69.1646 0)
       (effects (font (size 1.27 1.27)) (justify left top))
     )
-    (pin "V_Sen" output (at 180.34 66.04 180)
-      (effects (font (size 1.27 1.27)) (justify left))
-    )
-    (pin "Phase_Out" output (at 205.74 63.5 0)
-      (effects (font (size 1.27 1.27)) (justify right))
-    )
-    (pin "I_Sen" output (at 180.34 68.58 180)
+    (pin "Phase_Out" output (at 180.34 66.04 180)
       (effects (font (size 1.27 1.27)) (justify left))
     )
@@
       )
     )
+  )
+  (sheet (at 83.82 55.88) (size 25.4 10.16) (fields_autoplaced)
+    (stroke (width 0.1524) (type solid))
+    (fill (color 0 0 0 0.0000))
+    (property "Sheetname" "PSU" (at 83.82 55.1684 0)
+      (effects (font (size 1.27 1.27)) (justify left bottom))
+    )
+    (property "Sheetfile" "PSU.kicad_sch" (at 83.82 66.6246 0)
+      (effects (font (size 1.27 1.27)) (justify left top))
+    )
+    (instances
+      (project "BLDC-Controller"
+        (path "/3f98b8cc-f1be-42b2-9c23-c425b8147bc0" (page "6"))
+      )
+    )

Commit message: f
Other:
- note added: "- Battery = 3s to 6s"
- note added: "- Voltage input range = 10.5V to 25.2V"
- note removed: "- Battery = 2s to 6s"
- note removed: "- Voltage input range = 7V to 25.2V"
Changed lines of the file:
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@@
     (effects (font (size 1.27 1.27)) (justify left bottom))
   )
-  (text "- Voltage input range = 7V to 25.2V" (at 50.8 160.02 0)
+  (text "- Voltage input range = 10.5V to 25.2V" (at 50.8 160.02 0)
     (effects (font (size 1.27 1.27)) (justify left bottom))
   )
-  (text "- Battery = 2s to 6s" (at 50.8 157.48 0)
+  (text "- Battery = 3s to 6s" (at 50.8 157.48 0)
     (effects (font (size 1.27 1.27)) (justify left bottom))
   )

Commit message: Completed initial prototype.
Other:
- removed sheet PSU
- note added: "Figure 1: Hall sensor signal, back EMF, output torque and phase current"
- note added: "Source: https://ww1.microchip.com/downloads/en/Appnotes/00885a.pdf"

Commit message: Uploaded working software.
Other:
- note removed: "- Rated current = 50A"
- note removed: "- Voltage/current sensing for each phase"
- company: (none) -> Aria Tso
- title: (none) -> XE636 BLDC Motor Controller
Changed lines of the file:
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@@
 (kicad_sch (version 20230121) (generator eeschema)
   (paper "A4")
+  (title_block
+    (title "XE636 BLDC Motor Controller")
+    (date "2024-03-09")
+    (rev "V1.0")
+    (company "Aria Tso")
+  )
   (wire (pts (xy 45.72 25.4) (xy 55.88 25.4))
     (stroke (width 0) (type default))
@@
     )
   )
-  (text "- Voltage/current sensing for each phase" (at 20.32 101.6 0)
-    (effects (font (size 1.27 1.27)) (justify left bottom))
-  )
   (text "- Voltage input range = 10.5V to 25.2V" (at 20.32 96.52 0)
     (effects (font (size 1.27 1.27)) (justify left bottom))
@@
     (effects (font (size 1.27 1.27)) (justify left bottom))
   )
-  (text "- Rated current = 50A" (at 20.32 99.06 0)
-    (effects (font (size 1.27 1.27)) (justify left bottom))
-  )

Commit message: V2 started
Other:
- sheet MCU ports: added V_Sen_A, V_Sen_B, V_Sen_C, V_Sen_COM; removed Phase_Out_A, Phase_Out_B, Phase_Out_C
- sheet Phase A ports: added V_Sen, V_Sen_COM; removed Phase_Out
- sheet Phase B ports: added V_Sen, V_Sen_COM; removed Phase_Out
- sheet Phase C ports: added V_Sen, V_Sen_COM; removed Phase_Out
- note added: "- Rated current = 50A"
- note added: "- Voltage/current sensing for each phase"
- company: Aria Tso -> (none)
- title: XE636 BLDC Motor Controller -> (none)
Changed lines of the file:
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@@
 (kicad_sch (version 20230121) (generator eeschema)
   (paper "A4")
-  (title_block
-    (title "XE636 BLDC Motor Controller")
-    (date "2024-03-09")
-    (rev "V1.0")
-    (company "Aria Tso")
+  (junction (at 50.8 35.56) (diameter 0) (color 0 0 0 0)
+  )
+  (junction (at 50.8 58.42) (diameter 0) (color 0 0 0 0)
+  )
+  (wire (pts (xy 45.72 33.02) (xy 55.88 33.02))
+    (stroke (width 0) (type default))
+  )
+  (wire (pts (xy 45.72 35.56) (xy 50.8 35.56))
+    (stroke (width 0) (type default))
+  )
+  (wire (pts (xy 45.72 78.74) (xy 55.88 78.74))
+    (stroke (width 0) (type default))
   )
   (wire (pts (xy 45.72 25.4) (xy 55.88 25.4))
     (stroke (width 0) (type default))
   )
-  (wire (pts (xy 45.72 33.02) (xy 55.88 33.02))
-    (stroke (width 0) (type default))
-  )
-  (wire (pts (xy 45.72 78.74) (xy 55.88 78.74))
+  (wire (pts (xy 45.72 55.88) (xy 55.88 55.88))
+    (stroke (width 0) (type default))
+  )
+  (wire (pts (xy 50.8 35.56) (xy 55.88 35.56))
+    (stroke (width 0) (type default))
+  )
+  (wire (pts (xy 50.8 58.42) (xy 50.8 81.28))
     (stroke (width 0) (type default))
   )
@@
     (stroke (width 0) (type default))
   )
+  (wire (pts (xy 55.88 58.42) (xy 50.8 58.42))
+    (stroke (width 0) (type default))
+  )
   (wire (pts (xy 45.72 27.94) (xy 55.88 27.94))
     (stroke (width 0) (type default))
   )
-  (wire (pts (xy 45.72 55.88) (xy 55.88 55.88))
-    (stroke (width 0) (type default))
-  )
   (wire (pts (xy 45.72 73.66) (xy 55.88 73.66))
     (stroke (width 0) (type default))
@@
     (stroke (width 0) (type default))
   )
+  (wire (pts (xy 50.8 81.28) (xy 55.88 81.28))
+    (stroke (width 0) (type default))
+  )
   (wire (pts (xy 45.72 48.26) (xy 55.88 48.26))
+    (stroke (width 0) (type default))
+  )
+  (wire (pts (xy 50.8 58.42) (xy 50.8 35.56))
     (stroke (width 0) (type default))
   )
@@
     )
   )
+  (text "- Voltage/current sensing for each phase" (at 20.32 101.6 0)
+    (effects (font (size 1.27 1.27)) (justify left bottom))
+  )
   (text "- Voltage input range = 10.5V to 25.2V" (at 20.32 96.52 0)
     (effects (font (size 1.27 1.27)) (justify left bottom))
@@
     (effects (font (size 1.27 1.27)) (justify left bottom))
   )
-  (sheet (at 55.88 22.86) (size 25.4 12.7) (fields_autoplaced)
+  (text "- Rated current = 50A" (at 20.32 99.06 0)
+    (effects (font (size 1.27 1.27)) (justify left bottom))
+  )
+  (sheet (at 55.88 22.86) (size 25.4 15.24) (fields_autoplaced)
     (stroke (width 0.1524) (type solid))
     (fill (color 0 0 0 0.0000))
@@
       (effects (font (size 1.27 1.27)) (justify left bottom))
     )
-    (property "Sheetfile" "Phase.kicad_sch" (at 55.88 36.1446 0)
+    (property "Sheetfile" "Phase.kicad_sch" (at 55.88 38.6846 0)
       (effects (font (size 1.27 1.27)) (justify left top))
-    )
-    (pin "Phase_Out" output (at 55.88 33.02 180)
-      (effects (font (size 1.27 1.27)) (justify left))
     )
     (pin "HI" input (at 55.88 25.4 180)
@@
     )
     (pin "LI" input (at 55.88 27.94 180)
+      (effects (font (size 1.27 1.27)) (justify left))
+    )
+    (pin "V_Sen_COM" output (at 55.88 35.56 180)
+      (effects (font (size 1.27 1.27)) (justify left))
+    )
+    (pin "V_Sen" output (at 55.88 33.02 180)
       (effects (font (size 1.27 1.27)) (justify left))
     )
@@
     )
   )
-  (sheet (at 55.88 45.72) (size 25.4 12.7) (fields_autoplaced)
+  (sheet (at 55.88 45.72) (size 25.4 15.24) (fields_autoplaced)
     (stroke (width 0.1524) (type solid))
     (fill (color 0 0 0 0.0000))
@@
       (effects (font (size 1.27 1.27)) (justify left bottom))
     )
-    (property "Sheetfile" "Phase.kicad_sch" (at 55.88 59.0046 0)
+    (property "Sheetfile" "Phase.kicad_sch" (at 55.88 61.5446 0)
       (effects (font (size 1.27 1.27)) (justify left top))
-    )
-    (pin "Phase_Out" output (at 55.88 55.88 180)
-      (effects (font (size 1.27 1.27)) (justify left))
     )
     (pin "HI" input (at 55.88 48.26 180)
@@
     )
     (pin "LI" input (at 55.88 50.8 180)
+      (effects (font (size 1.27 1.27)) (justify left))
+    )
+    (pin "V_Sen_COM" output (at 55.88 58.42 180)
+      (effects (font (size 1.27 1.27)) (justify left))
+    )
+    (pin "V_Sen" output (at 55.88 55.88 180)
       (effects (font (size 1.27 1.27)) (justify left))
     )
@@
     )
   )
-  (sheet (at 55.88 68.58) (size 25.4 12.7) (fields_autoplaced)
+  (sheet (at 55.88 68.58) (size 25.4 15.24) (fields_autoplaced)
     (stroke (width 0.1524) (type solid))
     (fill (color 0 0 0 0.0000))
@@
       (effects (font (size 1.27 1.27)) (justify left bottom))
     )
-    (property "Sheetfile" "Phase.kicad_sch" (at 55.88 81.8646 0)
+    (property "Sheetfile" "Phase.kicad_sch" (at 55.88 84.4046 0)
       (effects (font (size 1.27 1.27)) (justify left top))
-    )
-    (pin "Phase_Out" output (at 55.88 78.74 180)
-      (effects (font (size 1.27 1.27)) (justify left))
     )
     (pin "HI" input (at 55.88 71.12 180)
@@
     )
     (pin "LI" input (at 55.88 73.66 180)
+      (effects (font (size 1.27 1.27)) (justify left))
+    )
+    (pin "V_Sen_COM" output (at 55.88 81.28 180)
+      (effects (font (size 1.27 1.27)) (justify left))
+    )
+    (pin "V_Sen" output (at 55.88 78.74 180)
       (effects (font (size 1.27 1.27)) (justify left))
     )
@@
     )
   )
-  (sheet (at 20.32 22.86) (size 25.4 58.42) (fields_autoplaced)
+  (sheet (at 20.32 22.86) (size 25.4 60.96) (fields_autoplaced)
     (stroke (width 0.1524) (type solid))
     (fill (color 0 0 0 0.0000))
@@
       (effects (font (size 1.27 1.27)) (justify left bottom))
     )
-    (property "Sheetfile" "MCU.kicad_sch" (at 20.32 81.8646 0)
+    (property "Sheetfile" "MCU.kicad_sch" (at 20.32 84.4046 0)
       (effects (font (size 1.27 1.27)) (justify left top))
     )
@@
       (effects (font (size 1.27 1.27)) (justify right))
     )
-    (pin "Phase_Out_C" input (at 45.72 78.74 0)
+    (pin "V_Sen_COM" input (at 45.72 35.56 0)
       (effects (font (size 1.27 1.27)) (justify right))
     )
-    (pin "Phase_Out_B" input (at 45.72 55.88 0)
+    (pin "V_Sen_B" input (at 45.72 55.88 0)
       (effects (font (size 1.27 1.27)) (justify right))
     )
-    (pin "Phase_Out_A" input (at 45.72 33.02 0)
+    (pin "V_Sen_A" input (at 45.72 33.02 0)
       (effects (font (size 1.27 1.27)) (justify right))
     )
+    (pin "V_Sen_C" input (at 45.72 78.74 0)
+      (effects (font (size 1.27 1.27)) (justify right))
+    )
